File: soc.kicad_sch (KiCad schematic)
At the start: 0 parts

Commit message: soc board
Parts:
- added U1: RK3568, RK3568:BGA-636_L19.0-W19.0-P0.65-BL, symbol RK3568:RK3568
Connections:
- new net CLK32K_IN: U1.AD23 (CLK32K_IN/CLK32K_OUT0/PCIE30X2_BUTTONRSTn/GPIO0_B0_u)
- new net CLK32K_OUT1: U1.E26 (CLK32K_OUT1/UART8_RX_M0/SPI1_CS1_M0/GPIO2_C6_d)
- new net DDR4_A0: U1.B6 (DDR4_A0/LPDDR4_CLKP_B/DDR3_A9/-/AC0)
- new net DDR4_A1: U1.F5 (DDR4_A1/-/DDR3_A2/-/AC1)
- new net DDR4_A10: U1.D6 (DDR4_A10/LPDDR4_CKE0_B/DDR3_A10/-/AC10)
- new net DDR4_A11: U1.C2 (DDR4_A11/LPDDR4_A0_A/DDR3_A7/LPDDR3_A8/AC11)
- new net DDR4_A12: U1.C4 (DDR4_A12/LPDDR4_A3_A/DDR3_BA2/-/AC12)
- new net DDR4_A13: U1.B8 (DDR4_A13/LPDDR4_A0_B/DDR3_A14/LPDDR3_A0/AC13)
- new net DDR4_A14_WEn: U1.C5 (DDR4_A14_WEn/LPDDR4_A4_A/DDR3_A15/LPDDR3_A5/AC14)
- new net DDR4_A15_CASn: U1.E4 (DDR4_A15_CASn/LPDDR4_A2_A/DDR3_A0/-/AC15)
- new net DDR4_A16_RASn: U1.D5 (DDR4_A16_RASn/LPDDR4_A5_A/DDR3_RASn/LPDDR3_A7/AC16)
- new net DDR4_A2: U1.B1 (DDR4_A2/LPDDR4_A1_A/DDR3_A4/LPDDR3_A6/AC2)
- new net DDR4_A3: U1.F4 (DDR4_A3/LPDDR4_CKE1_A/DDR3_A3/-/AC3)
- new net DDR4_A4: U1.D9 (DDR4_A4/LPDDR4_A3_B/DDR3_BA1/LPDDR3_A3/AC4)
- new net DDR4_A5: U1.B7 (DDR4_A5/LPDDR4_A5_B/DDR3_A11/LPDDR3_A2/AC5)
- new net DDR4_A6: U1.A7 (DDR4_A6/LPDDR4_A1_B/DDR3_A13/LPDDR3_A1/AC6)
- new net DDR4_A7: U1.A8 (DDR4_A7/LPDDR4_ODT0_CA_B/DDR3_A8/-/AC7)
- new net DDR4_A8: U1.C1 (DDR4_A8/LPDDR4_ODT0_CA_A/DDR3_A6/LPDDR3_A9/AC8)
- new net DDR4_A9: U1.A5 (DDR4_A9/LPDDR4_CLKN_B/DDR3_A5/-/AC9)
- new net DDR4_ACTn: U1.E6 (DDR4_ACTn/LPDDR4_CKE1_B/DDR3_CASn/-/AC17)
- new net DDR4_BA0: U1.E11 (DDR4_BA0/LPDDR4_A2_B/DDR3_A1/-/AC18)
- new net DDR4_BA1: U1.E9 (DDR4_BA1/LPDDR4_A4_B/DDR3_A12/LPDDR3_A4/AC19)
- new net DDR4_BG0: U1.F8 (DDR4_BG0/LPDDR4_ODT1_CA_B/DDR3_WEn/-/AC20)
- new net DDR4_BG1: U1.F7 (DDR4_BG1/LPDDR4_ODT1_CA_A/DDR3_BA0/-/AC21)
- new net DDR4_CKE: U1.B3 (DDR4_CKE/LPDDR4_CKE0_A/DDR3_CKE/LPDDR3_CKE/AC22)
- new net DDR4_CLKN: U1.A4 (DDR4_CLKN/LPDDR4_CLKN_A/DDR3_CLKN/LPDDR3_CLKN/AC24)
- new net DDR4_CLKP: U1.B4 (DDR4_CLKP/LPDDR4_CLKP_A/DDR3_CLKP/LPDDR3_CLKP/AC23)
- new net DDR4_CS0n: U1.A2 (DDR4_CS0n/LPDDR4_CS0n_A/DDR3_ODT1/LPDDR3_ODT0/AC25)
- new net DDR4_CS1n: U1.B2 (DDR4_CS1n/LPDDR4_CS1n_A/DDR3_CS1n/LPDDR3_ODT1/AC26)
- new net DDR4_ODT0: U1.E8 (DDR4_ODT0/LPDDR4_CS1n_B/DDR3_ODT0/LPDDR3_CS1n/AC27)
- new net DDR4_ODT1: U1.D8 (DDR4_ODT1/LPDDR4_CS0n_B/DDR3_CS0n/LPDDR3_CS0n/AC28)
- new net DDR4_RESETn: U1.F11 (DDR4_RESETn/LPDDR4_RESETn/DDR3_RESETn/AC29)
- new net DDR_DM0_A: U1.H5 (DDR_DM0_A/DDR4_DML_A/LPDDR4_DM0_A/DDR3_DM0/LPDDR3_DM1)
- new net DDR_DM0_B: U1.D14 (DDR_DM0_B/DDR4_DMU_B/LPDDR4_DM0_B/DDR3_DM2/LPDDR3_DM0)
- new net DDR_DM1_A: U1.J4 (DDR_DM1_A/DDR4_DMU_A/LPDDR4_DM1_A/DDR3_DM1/LPDDR3_DM3)
- new net DDR_DM1_B: U1.E17 (DDR_DM1_B/DDR4_DML_B/LPDDR4_DM1_B/DDR3_DM3/LPDDR3_DM2)
- new net DDR_DQ0_A: U1.F2 (DDR_DQ0_A/DDR4_DQL0_A/LPDDR4_DQ0_A/DDR3_DQ0/LPDDR3_DQ15)
- new net DDR_DQ0_B: U1.B10 (DDR_DQ0_B/DDR4_DQU7_B/LPDDR4_DQ0_B/DDR3_DQ16/LPDDR3_DQ1)
- new net DDR_DQ10_A: U1.L7 (DDR_DQ10_A/DDR4_DQU7_A/LPDDR4_DQ10_A/DDR3_DQ10/LPDDR3_DQ28)
- new net DDR_DQ10_B: U1.A17 (DDR_DQ10_B/DDR4_DQL4_B/LPDDR4_DQ10_B/DDR3_DQ26/LPDDR3_DQ22)
- new net DDR_DQ11_A: U1.L6 (DDR_DQ11_A/DDR4_DQU5_A/LPDDR4_DQ11_A/DDR3_DQ11/LPDDR3_DQ29)
- new net DDR_DQ11_B: U1.B18 (DDR_DQ11_B/DDR4_DQL6_B/LPDDR4_DQ11_B/DDR3_DQ27/LPDDR3_DQ23)
- new net DDR_DQ12_A: U1.K2 (DDR_DQ12_A/DDR4_DQU2_A/LPDDR4_DQ12_A/DDR3_DQ12/LPDDR3_DQ26)
- new net DDR_DQ12_B: U1.B13 (DDR_DQ12_B/DDR4_DQL7_B/LPDDR4_DQ12_B/DDR3_DQ28/LPDDR3_DQ16)
- new net DDR_DQ13_A: U1.J6 (DDR_DQ13_A/DDR4_DQU4_A/LPDDR4_DQ13_A/DDR3_DQ13/LPDDR3_DQ31)
- new net DDR_DQ13_B: U1.A13 (DDR_DQ13_B/DDR4_DQL5_B/LPDDR4_DQ13_B/DDR3_DQ29/LPDDR3_DQ17)
- new net DDR_DQ14_A: U1.J7 (DDR_DQ14_A/DDR4_DQU6_A/LPDDR4_DQ14_A/DDR3_DQ14/LPDDR3_DQ30)
- new net DDR_DQ14_B: U1.D17 (DDR_DQ14_B/DDR4_DQL1_B/LPDDR4_DQ14_B/DDR3_DQ30/LPDDR3_DQ20)
- new net DDR_DQ15_A: U1.L4 (DDR_DQ15_A/DDR4_DQU0_A/LPDDR4_DQ15_A/DDR3_DQ15/LPDDR3_DQ27)
- new net DDR_DQ15_B: U1.B14 (DDR_DQ15_B/DDR4_DQL3_B/LPDDR4_DQ15_B/DDR3_DQ31/LPDDR3_DQ21)
- new net DDR_DQ1_A: U1.E1 (DDR_DQ1_A/DDR4_DQL2_A/LPDDR4_DQ1_A/DDR3_DQ1/LPDDR3_DQ14)
- new net DDR_DQ1_B: U1.A9 (DDR_DQ1_B/DDR4_DQU5_B/LPDDR4_DQ1_B/DDR3_DQ17/LPDDR3_DQ5)
- new net DDR_DQ2_A: U1.E2 (DDR_DQ2_A/DDR4_DQL4_A/LPDDR4_DQ2_A/DDR3_DQ2/LPDDR3_DQ10)
- new net DDR_DQ2_B: U1.D12 (DDR_DQ2_B/DDR4_DQU3_B/LPDDR4_DQ2_B/DDR3_DQ18/LPDDR3_DQ6)
- new net DDR_DQ3_A: U1.D1 (DDR_DQ3_A/DDR4_DQL6_A/LPDDR4_DQ3_A/DDR3_DQ3/LPDDR3_DQ9)
- new net DDR_DQ3_B: U1.E12 (DDR_DQ3_B/DDR4_DQU1_B/LPDDR4_DQ3_B/DDR3_DQ19/LPDDR3_DQ4)
- new net DDR_DQ4_A: U1.J1 (DDR_DQ4_A/DDR4_DQL7_A/LPDDR4_DQ4_A/DDR3_DQ4/LPDDR3_DQ13)
- new net DDR_DQ4_B: U1.A12 (DDR_DQ4_B/DDR4_DQU0_B/LPDDR4_DQ4_B/DDR3_DQ20/LPDDR3_DQ2)
- new net DDR_DQ5_A: U1.J2 (DDR_DQ5_A/DDR4_DQL5_A/LPDDR4_DQ5_A/DDR3_DQ5/LPDDR3_DQ12)
- new net DDR_DQ5_B: U1.D15 (DDR_DQ5_B/DDR4_DQU6_B/LPDDR4_DQ5_B/DDR3_DQ21/LPDDR3_DQ3)
- new net DDR_DQ6_A: U1.H1 (DDR_DQ6_A/DDR4_DQL3_A/LPDDR4_DQ6_A/DDR3_DQ6/LPDDR3_DQ8)
- new net DDR_DQ6_B: U1.E15 (DDR_DQ6_B/DDR4_DQU4_B/LPDDR4_DQ6_B/DDR3_DQ22/LPDDR3_DQ7)
- new net DDR_DQ7_A: U1.H4 (DDR_DQ7_A/DDR4_DQL1_A/LPDDR4_DQ7_A/DDR3_DQ7/LPDDR3_DQ11)
- new net DDR_DQ7_B: U1.E14 (DDR_DQ7_B/DDR4_DQU2_B/LPDDR4_DQ7_B/DDR3_DQ23/LPDDR3_DQ0)
- new net DDR_DQ8_A: U1.M1 (DDR_DQ8_A/DDR4_DQU3_A/LPDDR4_DQ8_A/DDR3_DQ8/LPDDR3_DQ25)
- new net DDR_DQ8_B: U1.A16 (DDR_DQ8_B/DDR4_DQL0_B/LPDDR4_DQ8_B/DDR3_DQ24/LPDDR3_DQ18)
- new net DDR_DQ9_A: U1.N2 (DDR_DQ9_A/DDR4_DQU1_A/LPDDR4_DQ9_A/DDR3_DQ9/LPDDR3_DQ24)
- new net DDR_DQ9_B: U1.B17 (DDR_DQ9_B/DDR4_DQL2_B/LPDDR4_DQ9_B/DDR3_DQ25/LPDDR3_DQ19)
- new net DDR_DQS0N_A: U1.G2 (DDR_DQS0N_A/DDR4_DQSL_N_A/LPDDR4_DQS0N_A/DDR3_DQS0N/LPDDR3_DQS1N)
- new net DDR_DQS0N_B: U1.B11 (DDR_DQS0N_B/DDR4_DQSU_N_B/LPDDR4_DQS0N_B/DDR3_DQS2N/LPDDR3_DQS0N)
- new net DDR_DQS0P_A: U1.G1 (DDR_DQS0P_A/DDR4_DQSL_P_A/LPDDR4_DQS0P_A/DDR3_DQS0P/LPDDR3_DQS1P)
- new net DDR_DQS0P_B: U1.A11 (DDR_DQS0P_B/DDR4_DQSU_P_B/LPDDR4_DQS0P_B/DDR3_DQS2P/LPDDR3_DQS0P)
- new net DDR_DQS1N_A: U1.L1 (DDR_DQS1N_A/DDR4_DQSU_N_A/LPDDR4_DQS1N_A/DDR3_DQS1N/LPDDR3_DQS3N)
- new net DDR_DQS1N_B: U1.A15 (DDR_DQS1N_B/DDR4_DQSL_N_B/LPDDR4_DQS1N_B/DDR3_DQS3N/LPDDR3_DQS2N)
- new net DDR_DQS1P_A: U1.L2 (DDR_DQS1P_A/DDR4_DQSU_P_A/LPDDR4_DQS1P_A/DDR3_DQS1P/LPDDR3_DQS3P)
- new net DDR_DQS1P_B: U1.B15 (DDR_DQS1P_B/DDR4_DQSL_P_B/LPDDR4_DQS1P_B/DDR3_DQS3P/LPDDR3_DQS2P)
- new net DDR_ECC_DM: U1.P7 (DDR_ECC_DM)
- new net DDR_ECC_DQ0: U1.P5 (DDR_ECC_DQ0)
- new net DDR_ECC_DQ1: U1.M4 (DDR_ECC_DQ1)
- new net DDR_ECC_DQ2: U1.M5 (DDR_ECC_DQ2)
- new net DDR_ECC_DQ3: U1.R5 (DDR_ECC_DQ3)
- new net DDR_ECC_DQ4: U1.M7 (DDR_ECC_DQ4)
- new net DDR_ECC_DQ5: U1.R7 (DDR_ECC_DQ5)
- new net DDR_ECC_DQ6: U1.P4 (DDR_ECC_DQ6)
- new net DDR_ECC_DQ7: U1.R4 (DDR_ECC_DQ7)
- new net DDR_ECC_DQS_N: U1.P1 (DDR_ECC_DQS_N)
- new net DDR_ECC_DQS_P: U1.P2 (DDR_ECC_DQS_P)
- new net DDR_RZQ: U1.H7 (DDR_RZQ)
- new net DDR_VREFOUT: U1.P8 (DDR_VREFOUT)
- new net EDP_HPDIN: U1.AH7 (EDP_HPDIN_M0/SPDIF_TX_M2/SATA2_ACT_LED/PCIE30X2_PERSTn_M2/I2S3_LRCK_M1/GPIO4_C4_d)
- new net EDP_TX_AUXN: U1.M25 (EDP_TX_AUXN)
- new net EDP_TX_AUXP: U1.L25 (EDP_TX_AUXP)
- new net EDP_TX_AVDD_0V9: U1.M20 (EDP_TX_AVDD_0V9)
- new net EDP_TX_AVDD_1V8: U1.M22 (EDP_TX_AVDD_1V8)
- new net EDP_TX_D0N: U1.K27 (EDP_TX_D0N)
- new net EDP_TX_D0P: U1.J28 (EDP_TX_D0P)
- new net EDP_TX_D1N: U1.L27 (EDP_TX_D1N)
- new net EDP_TX_D1P: U1.K28 (EDP_TX_D1P)
- new net EDP_TX_D2N: U1.M27 (EDP_TX_D2N)
- new net EDP_TX_D2P: U1.L28 (EDP_TX_D2P)
- new net EDP_TX_D3N: U1.N27 (EDP_TX_D3N)
- new net EDP_TX_D3P: U1.M28 (EDP_TX_D3P)
- new net EMMC_CLKOUT: U1.A23 (EMMC_CLKOUT/FLASH_DQS/GPIO1_C5_d)
- new net EMMC_CMD: U1.B22 (EMMC_CMD/FLASH_WRn/GPIO1_C4_u)
- new net EMMC_D0: U1.A24 (EMMC_D0/FLASH_D0/GPIO1_B4_u)
- new net EMMC_D1: U1.C21 (EMMC_D1/FLASH_D1/GPIO1_B5_u)
- new net EMMC_D2: U1.B24 (EMMC_D2/FLASH_D2/GPIO1_B6_u)
- new net EMMC_D3: U1.D21 (EMMC_D3/FLASH_D3/GPIO1_B7_u)
- new net EMMC_D4: U1.A25 (EMMC_D4/FLASH_D4/GPIO1_C0_u)
- new net EMMC_D5: U1.E21 (EMMC_D5/FLASH_D5/GPIO1_C1_u)
- new net EMMC_D6: U1.E22 (EMMC_D6/FLASH_D6/GPIO1_C2_u)
- new net EMMC_D7: U1.B25 (EMMC_D7/FLASH_D7/GPIO1_C3_u)
- new net EMMC_DATA_STROBE: U1.A26 (EMMC_DATA_STROBE/FSPI_CS1n/FLASH_CLE/GPIO1_C6_d)
- new net EMMC_RSTn: U1.F20 (EMMC_RSTn/FSPI_D2/FLASH_WPn/GPIO1_C7_d)
- new net FLASH_VOL_SEL: U1.AG25 (FLASH_VOL_SEL/GPIO0_A7_u)
- new net FSPI_CLK: U1.A22 (FSPI_CLK/FLASH_ALE/GPIO1_D0_d)
- new net FSPI_CS0n: U1.C23 (FSPI_CS0n/FLASH_CS0n/GPIO1_D3_u)
- new net FSPI_D0: U1.C24 (FSPI_D0/FLASH_RDY/GPIO1_D1_u)
- new net FSPI_D1: U1.D23 (FSPI_D1/FLASH_RDn/GPIO1_D2_u)
- new net FSPI_D3: U1.A27 (FSPI_D3/FLASH_CS1n/GPIO1_D4_u)
- new net GMAC0_ETH_REFCLK: U1.G23 (I2S2_MCLK_M0/ETH0_REFCLKO_25M/UART7_RTSn_M0/SPI2_CLK_M0/GPIO2_C1_d)
- new net GMAC0_MCLKINOUT: U1.F25 (I2S2_SCLK_TX_M0/GMAC0_MCLKINOUT/UART7_CTSn_M0/SPI2_MISO_M0/GPIO2_C2_d)
- new net GMAC0_MDC: U1.H24 (I2S2_LRCK_TX_M0/GMAC0_MDC/UART9_RTSn_M0/SPI2_MOSI_M0/GPIO2_C3_d)
- new net GMAC0_MDIO: U1.H23 (I2S2_SDO_M0/GMAC0_MDIO/UART9_CTSn_M0/SPI2_CS0_M0/GPIO2_C4_d)
- new net GMAC0_RXD0: U1.F27 (GMAC0_RXD0/UART1_CTSn_M0/SPI1_MISO_M0/GPIO2_B6_u)
- new net GMAC0_RXD1: U1.H25 (I2S2_SCLK_RX_M0/GMAC0_RXD1/UART6_RTSn_M0/SPI1_MOSI_M0/GPIO2_B7_d)
- new net GMAC0_RXDV_CRS: U1.F24 (I2S2_LRCK_RX_M0/GMAC0_RXDV_CRS/UART6_CTSn_M0/SPI1_CS0_M0/GPIO2_C0_d)
- new net GMAC0_RXER: U1.F26 (I2S2_SDI_M0/GMAC0_RXER/UART8_TX_M0/SPI2_CS1_M0/GPIO2_C5_d)
- new net GMAC0_TXD0: U1.F28 (GMAC0_TXD0/UART1_RX_M0/GPIO2_B3_u)
- new net GMAC0_TXD1: U1.G27 (GMAC0_TXD1/UART1_TX_M0/GPIO2_B4_u)
- new net GMAC0_TXEN: U1.G28 (GMAC0_TXEN/UART1_RTSn_M0/SPI1_CLK_M0/GPIO2_B5_u)
- new net GND: U1.A1 (VSS_1), U1.A10 (VSS_4), U1.A14 (VSS_5), U1.A18 (VSS_6), U1.A28 (VSS_7), U1.A3 (VSS_2), U1.A6 (VSS_3), U1.AA12 (AVSS_24), U1.AA14 (AVSS_25), U1.AA15 (AVSS_26), U1.AA17 (AVSS_27), U1.AA23 (VSS_135), U1.AA24 (AVSS_28), U1.AA26 (AVSS_29), U1.AA4 (VSS_133), U1.AA9 (VSS_134), U1.AB11 (AVSS_30), U1.AB12 (AVSS_31), U1.AB14 (AVSS_32), U1.AB15 (AVSS_33), U1.AB17 (AVSS_34), U1.AB2 (VSS_136), U1.AB24 (TVSS), U1.AB6 (VSS_137), U1.AC11 (AVSS_36), U1.AC12 (AVSS_37), U1.AC15 (AVSS_38), U1.AC18 (AVSS_39), U1.AC25 (AVSS_40), U1.AC26 (AVSS_41), U1.AC9 (AVSS_35), U1.AD26 (AVSS_42), U1.AD3 (VSS_138), U1.AE14 (AVSS_43), U1.AE17 (AVSS_44), U1.AE20 (AVSS_45), U1.AE21 (VSS_140), U1.AE27 (AVSS_46), U1.AE28 (AVSS_47), U1.AE6 (VSS_139), U1.AF11 (AVSS_49), U1.AF12 (AVSS_50), U1.AF14 (AVSS_51), U1.AF15 (AVSS_52), U1.AF17 (AVSS_53), U1.AF18 (AVSS_54), U1.AF20 (AVSS_55), U1.AF21 (AVSS_56), U1.AF26 (VSS_142), U1.AF3 (VSS_141), U1.AF9 (AVSS_48), U1.AG18 (AVSS_57), U1.AG5 (VSS_143), U1.AH1 (VSS_144), U1.AH18 (AVSS_58), U1.AH23 (AVSS_59), U1.AH28 (VSS_146), U1.AH8 (VSS_145), U1.B12 (VSS_10), U1.B16 (VSS_11), U1.B23 (VSS_12), U1.B26 (VSS_13), U1.B5 (VSS_8), U1.B9 (VSS_9), U1.C11 (VSS_18), U1.C12 (VSS_19), U1.C14 (VSS_20), U1.C15 (VSS_21), U1.C17 (VSS_22), U1.C18 (VSS_23), U1.C25 (VSS_24), U1.C3 (VSS_14), U1.C6 (VSS_15), U1.C8 (VSS_16), U1.C9 (VSS_17), U1.D11 (VSS_27), U1.D2 (VSS_25), U1.D28 (VSS_28), U1.D3 (VSS_26), U1.E3 (VSS_29), U1.E7 (VSS_30), U1.F1 (VSS_31), U1.F12 (VSS_34), U1.F14 (VSS_35), U1.F15 (VSS_36), U1.F17 (VSS_37), U1.F3 (VSS_32), U1.F9 (VSS_33), U1.G11 (VSS_42), U1.G12 (VSS_43), U1.G14 (VSS_44), U1.G15 (VSS_45), U1.G17 (VSS_46), U1.G18 (VSS_47), U1.G24 (VSS_48), U1.G5 (VSS_38), U1.G6 (VSS_39), U1.G8 (VSS_40), U1.G9 (VSS_41), U1.H2 (VSS_49), U1.H3 (VSS_50), U1.H6 (VSS_51), U1.J17 (VSS_54), U1.J18 (VSS_55), U1.J20 (VSS_56), U1.J22 (VSS_57), U1.J26 (VSS_58), U1.J27 (AVSS_1), U1.J3 (VSS_52), U1.J5 (VSS_53), U1.J8 (DDR_AVSS), U1.K1 (VSS_59), U1.K11 (VSS_60), U1.K12 (VSS_61), U1.K13 (VSS_62), U1.K14 (VSS_63), U1.K19 (VSS_64), U1.L11 (VSS_68), U1.L13 (VSS_69), U1.L14 (VSS_70), U1.L19 (VSS_71), U1.L20 (VSS_72), U1.L21 (VSS_73), U1.L24 (AVSS_2), U1.L26 (AVSS_3), U1.L3 (VSS_65), U1.L5 (VSS_66), U1.L8 (VSS_67), U1.M11 (VSS_78), U1.M13 (VSS_79), U1.M14 (VSS_80), U1.M16 (VSS_81), U1.M18 (VSS_82), U1.M2 (VSS_74), U1.M21 (AVSS_4), U1.M26 (AVSS_5), U1.M3 (VSS_75), U1.M6 (VSS_76), U1.M8 (VSS_77), U1.N1 (VSS_83), U1.N11 (SYSPLL_AVSS), U1.N12 (VSS_84), U1.N14 (VSS_85), U1.N15 (VSS_86), U1.N17 (VSS_87), U1.N18 (VSS_88), U1.N28 (AVSS_6), U1.P12 (VSS_91), U1.P14 (VSS_92), U1.P15 (VSS_93), U1.P17 (VSS_94), U1.P21 (AVSS_7), U1.P26 (AVSS_8), U1.P3 (VSS_89), U1.P6 (VSS_90), U1.R10 (VSS_97), U1.R11 (VSS_98), U1.R14 (VSS_99), U1.R15 (VSS_100), U1.R17 (VSS_101), U1.R18 (VSS_102), U1.R19 (VSS_103), U1.R23 (AVSS_9), U1.R26 (AVSS_10), U1.R3 (VSS_95), U1.R6 (VSS_96), U1.T10 (VSS_104), U1.T11 (VSS_105), U1.T14 (VSS_106), U1.T15 (VSS_107), U1.T17 (VSS_108), U1.T18 (VSS_109), U1.T19 (VSS_110), U1.U1 (VSS_111), U1.U10 (VSS_115), U1.U14 (VSS_116), U1.U15 (VSS_117), U1.U16 (VSS_118), U1.U17 (VSS_119), U1.U18 (VSS_120), U1.U23 (AVSS_11), U1.U26 (AVSS_12), U1.U6 (VSS_112), U1.U7 (VSS_113), U1.U8 (VSS_114), U1.V13 (VSS_124), U1.V14 (AVSS_13), U1.V15 (AVSS_14), U1.V16 (AVSS_15), U1.V20 (PMUPLL_AVSS), U1.V22 (AVSS_16), U1.V23 (AVSS_17), U1.V26 (AVSS_18), U1.V3 (VSS_121), U1.V8 (VSS_122), U1.V9 (VSS_123), U1.W10 (VSS_125), U1.W11 (VSS_126), U1.W12 (VSS_127), U1.W13 (VSS_128), U1.W17 (AVSS_19), U1.Y11 (VSS_131), U1.Y12 (VSS_132), U1.Y18 (AVSS_20), U1.Y23 (AVSS_21), U1.Y24 (AVSS_22), U1.Y26 (AVSS_23), U1.Y8 (VSS_129), U1.Y9 (VSS_130)
- new net GPIO0_A3: U1.AA22 (GPIO0_A3_u)
- new net GPIO0_A5: U1.AF25 (SDMMC0_PWREN/SATA_MP_SWITCH/PCIE20_CLKREQn_M0/GPIO0_A5_d)
- new net GPIO0_A6: U1.AE24 (GPU_PWREN/SATA_CP_POD/PCIE30X2_CLKREQn_M0/GPIO0_A6_d)
- new net GPIO0_B2: U1.AB21 (I2C0_SDA/GPIO0_B2_u)
- new net GPIO0_B4: U1.AB20 (I2C1_SDA/CAN0_RX_M0/PCIE20_BUTTONRSTn/MCU_JTAG_TCK/GPIO0_B4_u)
- new net GPIO0_B5: U1.AC22 (I2C2_SCL_M0/SPI0_CLK_M0/PCIE20_WAKEn_M0/PWM1_M1/GPIO0_B5_u)
- new net GPIO0_B6: U1.AA20 (I2C2_SDA_M0/SPI0_MOSI_M0/PCIE20_PERSTn_M0/PWM2_M1/GPIO0_B6_u)
- new net GPIO0_B7: U1.AH26 (PWM0_M0/CPUAVS/GPIO0_B7_d)
- new net GPIO0_C2: U1.AG23 (PWM3_IR/EDP_HPDIN_M1/PCIE30X1_WAKEn_M0/MCU_JTAG_TMS/GPIO0_C2_d)
- new net GPIO0_C3: U1.AE23 (PWM4/VOP_PWM_M0/PCIE30X1_PERSTn_M0/MCU_JTAG_TRSTn/GPIO0_C3_d)
- new net GPIO0_C4: U1.AD21 (PWM5/SPI0_CS1_M0/UART0_RTSn/GPIO0_C4_d)
- new net GPIO0_C5: U1.AC21 (PWM6/SPI0_MISO_M0/PCIE30X2_WAKEn_M0/GPIO0_C5_d)
- new net GPIO0_C6: U1.AD20 (PWM7_IR/SPI0_CS0_M0/PCIE30X2_PERSTn_M0/GPIO0_C6_d)
- new net GPIO0_C7: U1.AH25 (HDMITX_CEC_M1/PWM0_M1/UART0_CTSn/GPIO0_C7_d)
- new net GPIO0_D3: U1.AE26 (GPIO0_D3_d)
- new net GPIO0_D4: U1.AB23 (GPIO0_D4_d)
- new net GPIO0_D5: U1.AD25 (GPIO0_D5_d)
- new net GPIO0_D6: U1.AC24 (GPIO0_D6_d)
- new net GPIO1_A2: U1.A19 (I2S1_MCLK_M0/UART3_RTSn_M0/SCR_CLK/PCIE30X1_PERSTn_M2/GPIO1_A2_d)
- new net GPIO1_A3: U1.B19 (I2S1_SCLK_TX_M0/UART3_CTSn_M0/SCR_IO/PCIE30X1_WAKEn_M2/ACODEC_DAC_CLK/GPIO1_A3_d)
- new net GPIO1_A4: U1.F18 (I2S1_SCLK_RX_M0/UART4_RX_M0/PDM_CLK1_M0/SPDIF_TX_M0/GPIO1_A4_d)
- new net GPIO1_A5: U1.A20 (I2S1_LRCK_TX_M0/UART4_RTSn_M0/SCR_RST/PCIE30X1_CLKREQn_M2/ACODEC_DAC_SYNC/GPIO1_A5_d)
- new net GPIO1_A6: U1.C20 (I2S1_LRCK_RX_M0/UART4_TX_M0/PDM_CLK0_M0/AUDIOPWM_ROUT_P/GPIO1_A6_d)
- new net GPIO1_A7: U1.B20 (I2S1_SDO0_M0/UART4_CTSn_M0/SCR_DET/AUDIOPWM_ROUT_N/ACODEC_DAC_DATAL/GPIO1_A7_d)
- new net GPIO1_B0: U1.D20 (I2S1_SDO1_M0/I2S1_SDI3_M0/PDM_SDI3_M0/PCIE20_CLKREQn_M2/ACODEC_DAC_DATAR/GPIO1_B0_d)
- new net GPIO1_B1: U1.E20 (I2S1_SDO2_M0/I2S1_SDI2_M0/PDM_SDI2_M0/PCIE20_WAKEn_M2/ACODEC_ADC_SYNC/GPIO1_B1_d)
- new net GPIO1_B2: U1.A21 (I2S1_SDO3_M0/I2S1_SDI1_M0/PDM_SDI1_M0/PCIE20_PERSTn_M2/GPIO1_B2_d)
- new net GPIO1_B3: U1.B21 (I2S1_SDI0_M0/PDM_SDI0_M0/GPIO1_B3_d)
- new net GPIO2_D0: U1.AG6 (LCDC_D0/VOP_BT656_D0_M0/SPI0_MISO_M1/PCIE20_CLKREQn_M1/I2S1_MCLK_M2/GPIO2_D0_d)
- new net GPIO2_D1: U1.AD7 (LCDC_D1/VOP_BT656_D1_M0/SPI0_MOSI_M1/PCIE20_WAKEn_M1/I2S1_SCLK_TX_M2/GPIO2_D1_d)
- new net GPIO2_D2: U1.AC8 (LCDC_D2/VOP_BT656_D2_M0/SPI0_CS0_M1/PCIE30X1_CLKREQn_M1/I2S1_LRCK_TX_M2/GPIO2_D2_d)
- new net GPIO2_D3: U1.AC7 (LCDC_D3/VOP_BT656_D3_M0/SPI0_CLK_M1/PCIE30X1_WAKEn_M1/I2S1_SDI0_M2/GPIO2_D3_d)
- new net GPIO2_D4: U1.AF5 (LCDC_D4/VOP_BT656_D4_M0/SPI2_CS1_M1/PCIE30X2_CLKREQn_M1/I2S1_SDI1_M2/GPIO2_D4_d)
- new net GPIO2_D5: U1.AF6 (LCDC_D5/VOP_BT656_D5_M0/SPI2_CS0_M1/PCIE30X2_WAKEn_M1/I2S1_SDI2_M2/GPIO2_D5_d)
- new net GPIO2_D6: U1.AD6 (LCDC_D6/VOP_BT656_D6_M0/SPI2_MOSI_M1/PCIE30X2_PERSTn_M1/I2S1_SDI3_M2/GPIO2_D6_d)
- new net GPIO2_D7: U1.AH5 (LCDC_D7/VOP_BT656_D7_M0/SPI2_MISO_M1/UART8_TX_M1/I2S1_SDO0_M2/GPIO2_D7_d)
- new net GPIO3_A0: U1.AH4 (LCDC_CLK/VOP_BT656_CLK_M0/SPI2_CLK_M1/UART8_RX_M1/I2S1_SDO1_M2/GPIO3_A0_d)
- new net GPIO3_A1: U1.AB8 (LCDC_D8/VOP_BT1120_D0/SPI1_CS0_M1/PCIE30X1_PERSTn_M1/SDMMC2_D0_M1/GPIO3_A1_d)
- new net GPIO3_A2: U1.AE5 (LCDC_D9/VOP_BT1120_D1/GMAC1_TXD2_M0/I2S3_MCLK_M0/SDMMC2_D1_M1/GPIO3_A2_d)
- new net GPIO3_A3: U1.AG4 (LCDC_D10/VOP_BT1120_D2/GMAC1_TXD3_M0/I2S3_SCLK_M0/SDMMC2_D2_M1/GPIO3_A3_d)
- new net GPIO3_A4: U1.AF4 (LCDC_D11/VOP_BT1120_D3/GMAC1_RXD2_M0/I2S3_LRCK_M0/SDMMC2_D3_M1/GPIO3_A4_d)
- new net GPIO3_A5: U1.AH3 (LCDC_D12/VOP_BT1120_D4/GMAC1_RXD3_M0/I2S3_SDO_M0/SDMMC2_CMD_M1/GPIO3_A5_d)
- new net GPIO3_A6: U1.AG3 (LCDC_D13/VOP_BT1120_CLK/GMAC1_TXCLK_M0/I2S3_SDI_M0/SDMMC2_CLK_M1/GPIO3_A6_d)
- new net GPIO3_A7: U1.AH2 (LCDC_D14/VOP_BT1120_D5/GMAC1_RXCLK_M0/SDMMC2_DET_M1/GPIO3_A7_d)
- new net GPIO3_B0: U1.AG2 (LCDC_D15/VOP_BT1120_D6/ETH1_REFCLKO_25M_M0/SDMMC2_PWREN_M1/GPIO3_B0_d)
- new net GPIO3_B1: U1.AG1 (LCDC_D16/VOP_BT1120_D7/GMAC1_RXD0_M0/UART4_RX_M1/PWM8_M0/GPIO3_B1_d)
- new net GPIO3_B2: U1.AF2 (LCDC_D17/VOP_BT1120_D8/GMAC1_RXD1_M0/UART4_TX_M1/PWM9_M0/GPIO3_B2_d)
- new net GPIO3_B3: U1.AF1 (LCDC_D18/VOP_BT1120_D9/GMAC1_RXDV_CRS_M0/I2C5_SCL_M0/PDM_SDI0_M2/GPIO3_B3_d)
- new net GPIO3_B4: U1.AE1 (LCDC_D19/VOP_BT1120_D10/GMAC1_RXER_M0/I2C5_SDA_M0/PDM_SDI1_M2/GPIO3_B4_d)
- new net GPIO3_B5: U1.AE2 (LCDC_D20/VOP_BT1120_D11/GMAC1_TXD0_M0/I2C3_SCL_M1/PWM10_M0/GPIO3_B5_d)
- new net GPIO3_B6: U1.AE3 (LCDC_D21/VOP_BT1120_D12/GMAC1_TXD1_M0/I2C3_SDA_M1/PWM11_IR_M0/GPIO3_B6_d)
- new net GPIO3_B7: U1.AD4 (LCDC_D22/PWM12_M0/GMAC1_TXEN_M0/UART3_TX_M1/PDM_SDI2_M2/GPIO3_B7_d)
- new net GPIO3_C0: U1.AD2 (LCDC_D23/PWM13_M0/GMAC1_MCLKINOUT_M0/UART3_RX_M1/PDM_SDI3_M2/GPIO3_C0_d)
- new net GPIO3_C1: U1.AD1 (LCDC_HSYNC/VOP_BT1120_D13/SPI1_MOSI_M1/PCIE20_PERSTn_M1/I2S1_SDO2_M2/GPIO3_C1_d)
- new net GPIO3_C2: U1.AA7 (LCDC_VSYNC/VOP_BT1120_D14/SPI1_MISO_M1/UART5_TX_M1/I2S1_SDO3_M2/GPIO3_C2_d)
- new net GPIO3_C3: U1.AC4 (LCDC_DEN/VOP_BT1120_D15/SPI1_CLK_M1/UART5_RX_M1/I2S1_SCLK_RX_M2/GPIO3_C3_d)
- new net GPIO3_C4: U1.AC3 (PWM14_M0/VOP_PWM_M1/GMAC1_MDC_M0/UART7_TX_M1/PDM_CLK1_M2/GPIO3_C4_d)
- new net GPIO3_C5: U1.AC2 (PWM15_IR_M0/SPDIF_TX_M1/GMAC1_MDIO_M0/UART7_RX_M1/I2S1_LRCK_RX_M2/GPIO3_C5_d)
- new net GPIO3_C6: U1.AC5 (CIF_D0/EBC_SDDO0/SDMMC2_D0_M0/I2S1_MCLK_M1/VOP_BT656_D0_M1/GPIO3_C6_d)
- new net GPIO3_C7: U1.AA6 (CIF_D1/EBC_SDDO1/SDMMC2_D1_M0/I2S1_SCLK_TX_M1/VOP_BT656_D1_M1/GPIO3_C7_d)
- new net GPIO3_D0: U1.AB5 (CIF_D2/EBC_SDDO2/SDMMC2_D2_M0/I2S1_LRCK_TX_M1/VOP_BT656_D2_M1/GPIO3_D0_d)
- new net GPIO3_D1: U1.AB1 (CIF_D3/EBC_SDDO3/SDMMC2_D3_M0/I2S1_SDO0_M1/VOP_BT656_D3_M1/GPIO3_D1_d)
- new net GPIO3_D2: U1.Y7 (CIF_D4/EBC_SDDO4/SDMMC2_CMD_M0/I2S1_SDI0_M1/VOP_BT656_D4_M1/GPIO3_D2_d)
- new net GPIO3_D3: U1.AC1 (CIF_D5/EBC_SDDO5/SDMMC2_CLK_M0/I2S1_SDI1_M1/VOP_BT656_D5_M1/GPIO3_D3_d)
- new net GPIO3_D4: U1.AA1 (CIF_D6/EBC_SDDO6/SDMMC2_DET_M0/I2S1_SDI2_M1/VOP_BT656_D6_M1/GPIO3_D4_d)
- new net GPIO3_D5: U1.AA5 (CIF_D7/EBC_SDDO7/SDMMC2_PWREN_M0/I2S1_SDI3_M1/VOP_BT656_D7_M1/GPIO3_D5_d)
- new net GPIO3_D6: U1.Y6 (CIF_D8/EBC_SDDO8/GMAC1_TXD2_M1/UART1_TX_M1/PDM_CLK0_M1/GPIO3_D6_d)
- new net GPIO3_D7: U1.Y5 (CIF_D9/EBC_SDDO9/GMAC1_TXD3_M1/UART1_RX_M1/PDM_SDI0_M1/GPIO3_D7_d)
- new net GPIO4_A0: U1.AA3 (CIF_D10/EBC_SDDO10/GMAC1_TXCLK_M1/PDM_CLK1_M1/GPIO4_A0_d)
- new net GPIO4_A1: U1.AA2 (CIF_D11/EBC_SDDO11/GMAC1_RXD2_M1/PDM_SDI1_M1/GPIO4_A1_d)
- new net GPIO4_A2: U1.Y4 (CIF_D12/EBC_SDDO12/GMAC1_RXD3_M1/UART7_TX_M2/PDM_SDI2_M1/GPIO4_A2_d)
- new net GPIO4_A3: U1.Y3 (CIF_D13/EBC_SDDO13/GMAC1_RXCLK_M1/UART7_RX_M2/PDM_SDI3_M1/GPIO4_A3_d)
- new net GPIO4_A4: U1.Y2 (CIF_D14/EBC_SDDO14/GMAC1_TXD0_M1/UART9_TX_M2/I2S2_LRCK_TX_M1/GPIO4_A4_d)
- new net GPIO4_A5: U1.Y1 (CIF_D15/EBC_SDDO15/GMAC1_TXD1_M1/UART9_RX_M2/I2S2_LRCK_RX_M1/GPIO4_A5_d)
- new net GPIO4_A6: U1.W2 (ISP_FLASHTRIGOUT/EBC_SDCE0/GMAC1_TXEN_M1/SPI3_CS0_M0/I2S1_SCLK_RX_M1/GPIO4_A6_d)
- new net GPIO4_A7: U1.W1 (CAM_CLKOUT0/EBC_SDCE1/GMAC1_RXD0_M1/SPI3_CS1_M0/I2S1_LRCK_RX_M1/GPIO4_A7_d)
- new net GPIO4_B0: U1.V7 (CAM_CLKOUT1/EBC_SDCE2/GMAC1_RXD1_M1/SPI3_MISO_M0/I2S1_SDO1_M1/GPIO4_B0_d)
- new net GPIO4_B1: U1.V2 (ISP_PRELIGHT_TRIG/EBC_SDCE3/GMAC1_RXDV_CRS_M1/I2S1_SDO2_M1/GPIO4_B1_d)
- new net GPIO4_B2: U1.V4 (I2C4_SDA_M0/EBC_VCOM/GMAC1_RXER_M1/SPI3_MOSI_M0/I2S2_SDI_M1/GPIO4_B2_d)
- new net GPIO4_B3: U1.V1 (I2C4_SCL_M0/EBC_GDOE/ETH1_REFCLKO_25M_M1/SPI3_CLK_M0/I2S2_SDO_M1/GPIO4_B3_d)
- new net GPIO4_B4: U1.V6 (I2C2_SDA_M1/EBC_GDSP/CAN2_RX_M0/ISP_FLASH_TRIGIN/VOP_BT656_CLK_M1/GPIO4_B4_d)
- new net GPIO4_B5: U1.V5 (I2C2_SCL_M1/EBC_SDSHR/CAN2_TX_M0/I2S1_SDO3_M1/GPIO4_B5_d)
- new net GPIO4_B6: U1.U5 (CIF_HREF/EBC_SDLE/GMAC1_MDC_M1/UART1_RTSn_M1/I2S2_MCLK_M1/GPIO4_B6_d)
- new net GPIO4_B7: U1.U4 (CIF_VSYNC/EBC_SDOE/GMAC1_MDIO_M1/I2S2_SCLK_TX_M1/GPIO4_B7_d)
- new net GPIO4_C0: U1.U3 (CIF_CLKOUT/EBC_GDCLK/PWM11_IR_M1/GPIO4_C0_d)
- new net GPIO4_C1: U1.U2 (CIF_CLKIN/EBC_SDCLK/GMAC1_MCLKINOUT_M1/UART1_CTSn_M1/I2S2_SCLK_RX_M1/GPIO4_C1_d)
- new net GPIO4_C2: U1.AF8 (PWM14_M1/SPI3_CLK_M1/CAN1_RX_M1/PCIE30X2_CLKREQn_M2/I2S3_MCLK_M1/GPIO4_C2_d)
- new net GPIO4_C3: U1.AA11 (PWM15_IR_M1/SPI3_MOSI_M1/CAN1_TX_M1/PCIE30X2_WAKEn_M2/I2S3_SCLK_M1/GPIO4_C3_d)
- new net GPIO4_C5: U1.AD8 (PWM12_M1/SPI3_MISO_M1/SATA1_ACT_LED/UART9_TX_M1/I2S3_SDO_M1/GPIO4_C5_d)
- new net GPIO4_C6: U1.AE8 (PWM13_M1/SPI3_CS0_M1/SATA0_ACT_LED/UART9_RX_M1/I2S3_SDI_M1/GPIO4_C6_d)
- new net GPIO4_D2: U1.AB9 (GPIO4_D2_d)
- new net HDMITX_CEC: U1.AH6 (HDMITX_CEC_M0/SPI3_CS1_M1/GPIO4_D1_u)
- new net HDMITX_SCL: U1.AG8 (HDMITX_SCL/I2C5_SCL_M1/GPIO4_C7_u)
- new net HDMITX_SDA: U1.AG7 (HDMITX_SDA/I2C5_SDA_M1/GPIO4_D0_u)
- new net HDMI_TX_AVDD_0V9: U1.V17 (HDMI_TX_AVDD_0V9_1), U1.V18 (HDMI_TX_AVDD_0V9_2)
- new net HDMI_TX_AVDD_1V8: U1.W18 (HDMI_TX_AVDD_1V8)
- new net HDMI_TX_CLKN: U1.AG19 (HDMI_TX_CLKN)
- new net HDMI_TX_CLKP: U1.AH19 (HDMI_TX_CLKP)
- new net HDMI_TX_D0N: U1.AH20 (HDMI_TX_D0N)
- new net HDMI_TX_D0P: U1.AG20 (HDMI_TX_D0P)
- new net HDMI_TX_D1N: U1.AH21 (HDMI_TX_D1N)
- new net HDMI_TX_D1P: U1.AG21 (HDMI_TX_D1P)
- new net HDMI_TX_D2N: U1.AH22 (HDMI_TX_D2N)
- new net HDMI_TX_D2P: U1.AG22 (HDMI_TX_D2P)
- new net HDMI_TX_HPDIN: U1.AB18 (HDMI_TX_HPDIN)
- new net HDMI_TX_REXT: U1.AA18 (HDMI_TX_REXT)
- new net I2C0_SCL: U1.AF24 (I2C0_SCL/GPIO0_B1_u)
- new net I2C1_SCL: U1.AG24 (I2C1_SCL/CAN0_TX_M0/PCIE30X1_BUTTONRSTn/MCU_JTAG_TDO/GPIO0_B3_u)
- new net I2C3_SCL: U1.E18 (I2C3_SCL_M0/UART3_TX_M0/CAN1_TX_M0/AUDIOPWM_LOUT_N/ACODEC_ADC_CLK/GPIO1_A1_u)
- new net I2C3_SDA: U1.D18 (I2C3_SDA_M0/UART3_RX_M0/CAN1_RX_M0/AUDIOPWM_LOUT_P/ACODEC_ADC_DATA/GPIO1_A0_u)
- new net MIPI_CSI_RX_AVDD_0V9: U1.W14 (MIPI_CSI_RX_AVDD_0V9)
- new net MIPI_CSI_RX_AVDD_1V8: U1.Y14 (MIPI_CSI_RX_AVDD_1V8)
- new net MIPI_CSI_RX_CLK0N: U1.AH10 (MIPI_CSI_RX_CLK0N)
- new net MIPI_CSI_RX_CLK0P: U1.AG10 (MIPI_CSI_RX_CLK0P)
- new net MIPI_CSI_RX_CLK1N: U1.AH9 (MIPI_CSI_RX_CLK1N)
- new net MIPI_CSI_RX_CLK1P: U1.AG9 (MIPI_CSI_RX_CLK1P)
- new net MIPI_CSI_RX_D0N: U1.AH12 (MIPI_CSI_RX_D0N)
- new net MIPI_CSI_RX_D0P: U1.AG12 (MIPI_CSI_RX_D0P)
- new net MIPI_CSI_RX_D1N: U1.AH11 (MIPI_CSI_RX_D1N)
- new net MIPI_CSI_RX_D1P: U1.AG11 (MIPI_CSI_RX_D1P)
- new net MIPI_CSI_RX_D2N: U1.AD11 (MIPI_CSI_RX_D2N)
- new net MIPI_CSI_RX_D2P: U1.AE11 (MIPI_CSI_RX_D2P)
- new net MIPI_CSI_RX_D3N: U1.AE9 (MIPI_CSI_RX_D3N)
- new net MIPI_CSI_RX_D3P: U1.AD9 (MIPI_CSI_RX_D3P)
- new net MIPI_DSI_TX0_AVDD_0V9: U1.W16 (MIPI_DSI_TX0/LVDS_TX0_AVDD_0V9)
- new net MIPI_DSI_TX0_AVDD_1V8: U1.Y17 (MIPI_DSI_TX0/LVDS_TX0_AVDD_1V8)
- new net MIPI_DSI_TX0_CLKN: U1.AG15 (MIPI_DSI_TX0_CLKN/LVDS_TX0_CLKN)
- new net MIPI_DSI_TX0_CLKP: U1.AH15 (MIPI_DSI_TX0_CLKP/LVDS_TX0_CLKP)
- new net MIPI_DSI_TX0_D0N: U1.AG17 (MIPI_DSI_TX0_D0N/LVDS_TX0_D0N)
- new net MIPI_DSI_TX0_D0P: U1.AH17 (MIPI_DSI_TX0_D0P/LVDS_TX0_D0P)
- new net MIPI_DSI_TX0_D1N: U1.AG16 (MIPI_DSI_TX0_D1N/LVDS_TX0_D1N)
- new net MIPI_DSI_TX0_D1P: U1.AH16 (MIPI_DSI_TX0_D1P/LVDS_TX0_D1P)
- new net MIPI_DSI_TX0_D2N: U1.AG14 (MIPI_DSI_TX0_D2N/LVDS_TX0_D2N)
- new net MIPI_DSI_TX0_D2P: U1.AH14 (MIPI_DSI_TX0_D2P/LVDS_TX0_D2P)
- new net MIPI_DSI_TX0_D3N: U1.AG13 (MIPI_DSI_TX0_D3N/LVDS_TX0_D3N)
- new net MIPI_DSI_TX0_D3P: U1.AH13 (MIPI_DSI_TX0_D3P/LVDS_TX0_D3P)
- new net MIPI_DSI_TX1_AVDD_0V9: U1.W15 (MIPI_DSI_TX1_AVDD_0V9)
- new net MIPI_DSI_TX1_AVDD_1V8: U1.Y15 (MIPI_DSI_TX1_AVDD_1V8)
- new net MIPI_DSI_TX1_CLKN: U1.AE15 (MIPI_DSI_TX1_CLKN)
- new net MIPI_DSI_TX1_CLKP: U1.AD15 (MIPI_DSI_TX1_CLKP)
- new net MIPI_DSI_TX1_D0N: U1.AE18 (MIPI_DSI_TX1_D0N)
- new net MIPI_DSI_TX1_D0P: U1.AD18 (MIPI_DSI_TX1_D0P)
- new net MIPI_DSI_TX1_D1N: U1.AC17 (MIPI_DSI_TX1_D1N)
- new net MIPI_DSI_TX1_D1P: U1.AD17 (MIPI_DSI_TX1_D1P)
- new net MIPI_DSI_TX1_D2N: U1.AC14 (MIPI_DSI_TX1_D2N)
- new net MIPI_DSI_TX1_D2P: U1.AD14 (MIPI_DSI_TX1_D2P)
- new net MIPI_DSI_TX1_D3N: U1.AE12 (MIPI_DSI_TX1_D3N)
- new net MIPI_DSI_TX1_D3P: U1.AD12 (MIPI_DSI_TX1_D3P)
- new net MULTI_PHY0_REFCLKN: U1.R25 (MULTI_PHY0_REFCLKN)
- new net MULTI_PHY0_REFCLKP: U1.R24 (MULTI_PHY0_REFCLKP)
- new net MULTI_PHY1_REFCLKN: U1.U24 (MULTI_PHY1_REFCLKN)
- new net MULTI_PHY1_REFCLKP: U1.U25 (MULTI_PHY1_REFCLKP)
- new net MULTI_PHY_AVDD_0V9: U1.R20 (MULTI_PHY_AVDD_0V9_1), U1.R21 (MULTI_PHY_AVDD_0V9_2)
- new net MULTI_PHY_AVDD_1V8: U1.R22 (MULTI_PHY_AVDD_1V8)
- new net OTP_VCC18: U1.H20 (OTP_VCC18)
- new net PCIE20_REFCLKN: U1.V25 (PCIE20_REFCLKN)
- new net PCIE20_REFCLKP: U1.V24 (PCIE20_REFCLKP)
- new net PCIE20_RXN: U1.Y28 (PCIE20_RXN/SATA2_RXN/QSGMII_RXN_M1)
- new net PCIE20_RXP: U1.Y27 (PCIE20_RXP/SATA2_RXP/QSGMII_RXP_M1)
- new net PCIE20_TXN: U1.W28 (PCIE20_TXN/SATA2_TXN/QSGMII_TXN_M1)
- new net PCIE20_TXP: U1.W27 (PCIE20_TXP/SATA2_TXP/QSGMII_TXP_M1)
- new net PCIE30_AVDD_0V9: U1.U20 (PCIE30_AVDD_0V9_2), U1.U21 (PCIE30_AVDD_0V9_1)
- new net PCIE30_AVDD_1V8: U1.U22 (PCIE30_AVDD_1V8)
- new net PCIE30_REFCLKN_IN: U1.AA25 (PCIE30_REFCLKN_IN)
- new net PCIE30_REFCLKP_IN: U1.Y25 (PCIE30_REFCLKP_IN)
- new net PCIE30_RESREF: U1.U19 (PCIE30_RESREF)
- new net PCIE30_RX0N: U1.AC27 (PCIE30_RX0N)
- new net PCIE30_RX0P: U1.AC28 (PCIE30_RX0P)
- new net PCIE30_RX1N: U1.AD27 (PCIE30_RX1N)
- new net PCIE30_RX1P: U1.AD28 (PCIE30_RX1P)
- new net PCIE30_TX0N: U1.AA27 (PCIE30_TX0N)
- new net PCIE30_TX0P: U1.AA28 (PCIE30_TX0P)
- new net PCIE30_TX1N: U1.AB27 (PCIE30_TX1N)
- new net PCIE30_TX1P: U1.AB28 (PCIE30_TX1P)
- new net PMIC_SLEEP: U1.AG28 (PMIC_SLEEP/TSADC_SHUT_M1/GPIO0_A2_d)
- new net PMUIO1: U1.Y20 (PMUIO1)
- new net PMUIO2: U1.W19 (PMUIO2)
- new net PMUPLL_AVDD_0V9: U1.V21 (PMUPLL_AVDD_0V9)
- new net PMUPLL_AVDD_1V8: U1.Y21 (PMUPLL_AVDD_1V8)
- new net PMU_VDD_LOGIC_0V9: U1.V19 (PMU_VDD_LOGIC_0V9)
- new net REFCLK_OUT: U1.AG27 (REFCLK_OUT/GPIO0_A0_d)
- new net SARADC_AVDD_1V8: U1.H22 (SARADC_AVDD_1V8)
- new net SARADC_VIN0: U1.B27 (SARADC_VIN0)
- new net SARADC_VIN1: U1.C26 (SARADC_VIN1)
- new net SARADC_VIN2: U1.D24 (SARADC_VIN2)
- new net SARADC_VIN3: U1.E23 (SARADC_VIN3)
- new net SARADC_VIN4: U1.G21 (SARADC_VIN4)
- new net SARADC_VIN5: U1.F22 (SARADC_VIN5)
- new net SARADC_VIN6: U1.G20 (SARADC_VIN6)
- new net SARADC_VIN7: U1.F21 (SARADC_VIN7)
- new net SDMMC0_CLK: U1.H28 (SDMMC0_CLK/TEST_CLKOUT/UART5_TX_M0/CAN0_RX_M1/GPIO2_A2_d)
- new net SDMMC0_CMD: U1.H27 (SDMMC0_CMD/PWM10_M1/UART5_RX_M0/CAN0_TX_M1/GPIO2_A1_u)
- new net SDMMC0_D0: U1.J25 (SDMMC0_D0/UART2_TX_M1/UART6_TX_M1/PWM8_M1/GPIO1_D5_u)
- new net SDMMC0_D1: U1.J24 (SDMMC0_D1/UART2_RX_M1/UART6_RX_M1/PWM9_M1/GPIO1_D6_u)
- new net SDMMC0_D2: U1.H26 (SDMMC0_D2/ARMJTAG_TCK/UART5_CTSn_M0/GPIO1_D7_u)
- new net SDMMC0_D3: U1.J23 (SDMMC0_D3/ARMJTAG_TMS/UART5_RTSn_M0/GPIO2_A0_u)
- new net SDMMC0_DET: U1.Y22 (SDMMC0_DET/SATA_CP_DET/PCIE30X1_CLKREQn_M0/GPIO0_A4_u)
- new net SDMMC1_CLK: U1.D27 (SDMMC1_CLK/GMAC0_TXCLK/UART9_TX_M0/GPIO2_B0_d)
- new net SDMMC1_CMD: U1.C28 (SDMMC1_CMD/GMAC0_TXD3/UART9_RX_M0/GPIO2_A7_u)
- new net SDMMC1_D0: U1.E27 (SDMMC1_D0/GMAC0_RXD2/UART6_RX_M0/GPIO2_A3_u)
- new net SDMMC1_D1: U1.E28 (SDMMC1_D1/GMAC0_RXD3/UART6_TX_M0/GPIO2_A4_u)
- new net SDMMC1_D2: U1.B28 (SDMMC1_D2/GMAC0_RXCLK/UART7_RX_M0/GPIO2_A5_u)
- new net SDMMC1_D3: U1.C27 (SDMMC1_D3/GMAC0_TXD2/UART7_TX_M0/GPIO2_A6_u)
- new net SDMMC1_DET: U1.E25 (SDMMC1_DET/I2C4_SCL_M1/UART8_CTSn_M0/CAN2_TX_M1/GPIO2_B2_u)
- new net SDMMC1_PWREN: U1.D26 (SDMMC1_PWREN/I2C4_SDA_M1/UART8_RTSn_M0/CAN2_RX_M1/GPIO2_B1_d)
- new net SYSPLL_AVDD_0V9: U1.P11 (SYSPLL_AVDD_0V9)
- new net SYSPLL_AVDD_1V8: U1.N10 (SYSPLL_AVDD_1V8)
- new net TSADC_SHUT: U1.AG26 (TSADC_SHUT_M0/TSADC_SHUT_ORG/GPIO0_A1_z)
- new net UART0_RX: U1.AD22 (PWM1_M0/GPUAVS/UART0_RX/GPIO0_C0_d)
- new net UART0_TX: U1.AF23 (PWM2_M0/NPUAVS/UART0_TX/MCU_JTAG_TDI/GPIO0_C1_d)
- new net UART2_RX: U1.AC20 (UART2_RX_M0/GPIO0_D0_u)
- new net UART2_TX: U1.AH24 (UART2_TX_M0/GPIO0_D1_u)
- new net USB2_AVDD_0V9: U1.R8 (USB2_AVDD_0V9)
- new net USB2_AVDD_1V8: U1.P9 (USB2_AVDD_1V8)
- new net USB2_AVDD_3V3: U1.P10 (USB2_AVDD_3V3)
- new net USB2_HOST2_DM: U1.R1 (USB2_HOST2_DM)
- new net USB2_HOST2_DP: U1.R2 (USB2_HOST2_DP)
- new net USB2_HOST3_DM: U1.T1 (USB2_HOST3_DM)
- new net USB2_HOST3_DP: U1.T2 (USB2_HOST3_DP)
- new net USB3_AVDD_0V9: U1.P22 (USB3_AVDD_0V9)
- new net USB3_AVDD_1V8: U1.P23 (USB3_AVDD_1V8)
- new net USB3_AVDD_3V3: U1.M23 (USB3_AVDD_3V3)
- new net USB3_HOST1_DM: U1.P25 (USB3_HOST1_DM)
- new net USB3_HOST1_DP: U1.P24 (USB3_HOST1_DP)
- new net USB3_HOST1_SSRXN: U1.U27 (USB3_HOST1_SSRXN/SATA1_RXN/QSGMII_RXN_M0)
- new net USB3_HOST1_SSRXP: U1.U28 (USB3_HOST1_SSRXP/SATA1_RXP/QSGMII_RXP_M0)
- new net USB3_HOST1_SSTXN: U1.V27 (USB3_HOST1_SSTXN/SATA1_TXN/QSGMII_TXN_M0)
- new net USB3_HOST1_SSTXP: U1.V28 (USB3_HOST1_SSTXP/SATA1_TXP/QSGMII_TXP_M0)
- new net USB3_OTG0_DM: U1.P28 (USB3_OTG0_DM)
- new net USB3_OTG0_DP: U1.P27 (USB3_OTG0_DP)
- new net USB3_OTG0_ID: U1.L23 (USB3_OTG0_ID)
- new net USB3_OTG0_SSRXN: U1.R27 (USB3_OTG0_SSRXN/SATA0_RXN)
- new net USB3_OTG0_SSRXP: U1.R28 (USB3_OTG0_SSRXP/SATA0_RXP)
- new net USB3_OTG0_SSTXN: U1.T27 (USB3_OTG0_SSTXN/SATA0_TXN)
- new net USB3_OTG0_SSTXP: U1.T28 (USB3_OTG0_SSTXP/SATA0_TXP)
- new net USB3_OTG0_VBUSDET: U1.M24 (USB3_OTG0_VBUSDET)
- new net VCCIO1: U1.H17 (VCCIO1)
- new net VCCIO2: U1.H18 (VCCIO2)
- new net VCCIO3: U1.L22 (VCCIO3)
- new net VCCIO4: U1.J21 (VCCIO4)
- new net VCCIO5: U1.V10 (VCCIO5_1), U1.V11 (VCCIO5_2)
- new net VCCIO6: U1.R9 (VCCIO6_1), U1.U9 (VCCIO6_2)
- new net VCCIO7: U1.V12 (VCCIO7)
- new net VCC_DDR: U1.H11 (DDRPHY_VDDQ_2), U1.H12 (DDRPHY_VDDQ_3), U1.H14 (DDRPHY_VDDQ_4), U1.H15 (DDRPHY_VDDQ_5), U1.H9 (DDRPHY_VDDQ_1), U1.J11 (DDRPHY_VDDQL_1), U1.J12 (DDRPHY_VDDQL_2), U1.J14 (DDRPHY_VDDQL_3), U1.J9 (DDRPHY_VDDQ_6), U1.K10 (DDRPHY_VDDQL_4), U1.L10 (DDRPHY_VDDQL_5), U1.L9 (DDRPHY_VDDQ_7), U1.M10 (DDRPHY_VDDQL_6), U1.M9 (DDRPHY_VDDQ_8)
- new net VDD_CPU: U1.J15 (VDD_CPU_1), U1.K15 (VDD_CPU_2), U1.K16 (VDD_CPU_3), U1.K17 (VDD_CPU_4), U1.K18 (VDD_CPU_5), U1.L15 (VDD_CPU_6), U1.L16 (VDD_CPU_7), U1.L17 (VDD_CPU_8), U1.L18 (VDD_CPU_9), U1.M15 (VDD_CPU_COM), U1.M17 (VDD_CPU_10)
- new net VDD_GPU: U1.R13 (VDD_GPU_1), U1.T13 (VDD_GPU_2), U1.U11 (VDD_GPU_3), U1.U12 (VDD_GPU_4), U1.U13 (VDD_GPU_5)
- new net VDD_LOGIC: U1.L12 (VDD_LOGIC_1), U1.M12 (VDD_LOGIC_2), U1.N13 (VDD_LOGIC_3), U1.N16 (VDD_LOGIC_4), U1.P13 (VDD_LOGIC_5), U1.P16 (VDD_LOGIC_6), U1.R12 (VDD_LOGIC_7), U1.R16 (VDD_LOGIC_8), U1.T12 (VDD_LOGIC_9), U1.T16 (VDD_LOGIC_10)
- new net VDD_NPU: U1.M19 (VDD_NPU_1), U1.N19 (VDD_NPU_2), U1.P18 (VDD_NPU_3), U1.P19 (VDD_NPU_4), U1.P20 (VDD_NPU_5)
- new net XIN24M: U1.AF28 (XIN24M)
- new net XOUT24M: U1.AF27 (XOUT24M)
- new net nPOR: U1.AH27 (nPOR_u)
