File: soc.kicad_sch (KiCad schematic)
At the start: 1 part, among them U1 RK3568

Commit message: display sheet
Other:
- title: (none) -> RK3506 SoC
Changed lines of the file:
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@@
 	(generator_version "10.0")
 	(paper "A0" portrait)
+	(title_block
+		(title "RK3506 SoC")
+	)
 	(no_connect
 		(at 572.77 251.46)
