File: soc.kicad_sch (KiCad schematic)
At the start: 1 part, among them U1 RK3568

Commit message: root sheet changes
Parts:
- renumbered U1 to U2
Changed lines of the file:
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@@
 		(in_pos_files yes)
 		(dnp no)
-		(property "Reference" "U1"
+		(property "Reference" "U2"
 			(at 420.37 187.96 0)
 			(show_name no)
@@
 				)
 				(path "/6ade62f6-9cb2-4783-8048-f18138ca0ff8/d3c630df-b147-44f4-bec8-a7b2c063ed94"
-					(reference "U1")
+					(reference "U2")
 					(unit 1)
 				)
