File: ddr_memory.kicad_sch (KiCad schematic)
At the start: 0 parts

Commit message: fixed netclasses
Parts:
- added C1, C11, C6: 10uF, symbol Device:C
- added C10, C12, C13, C14, C15, C2, C3, C4, C5, C7, C8, C9: 100nF, symbol Device:C
- added R1, R2: 240, symbol Device:R
- added U1: K4UCE3Q4AB-MGCL, K4UCE3Q4AB-MGCL:FBGA-200_L15.0-W10.0-BL_RS512M32LO4D1BDS-53BT, symbol K4UCE3Q4AB-MGCL:K4UCE3Q4AB-MGCL
Connections:
- new net DDR_DM0_A: U1.C3 (DMI0_a)
- new net DDR_DM0_B: U1.Y3 (DMI0_b)
- new net DDR_DM1_A: U1.C10 (DMI1_a)
- new net DDR_DM1_B: U1.Y10 (DMI1_b)
- new net DDR_DQ0_A: U1.B2 (DQ0_a)
- new net DDR_DQ0_B: U1.AA2 (DQ0_b)
- new net DDR_DQ10_A: U1.E11 (DQ10_a)
- new net DDR_DQ10_B: U1.V11 (DQ10_b)
- new net DDR_DQ11_A: U1.F11 (DQ11_a)
- new net DDR_DQ11_B: U1.U11 (DQ11_b)
- new net DDR_DQ12_A: U1.F9 (DQ12_a)
- new net DDR_DQ12_B: U1.U9 (DQ12_b)
- new net DDR_DQ13_A: U1.E9 (DQ13_a)
- new net DDR_DQ13_B: U1.V9 (DQ13_b)
- new net DDR_DQ14_A: U1.C9 (DQ14_a)
- new net DDR_DQ14_B: U1.Y9 (DQ14_b)
- new net DDR_DQ15_A: U1.B9 (DQ15_a)
- new net DDR_DQ15_B: U1.AA9 (DQ15_b)
- new net DDR_DQ1_A: U1.C2 (DQ1_a)
- new net DDR_DQ1_B: U1.Y2 (DQ1_b)
- new net DDR_DQ2_A: U1.E2 (DQ2_a)
- new net DDR_DQ2_B: U1.V2 (DQ2_b)
- new net DDR_DQ3_A: U1.F2 (DQ3_a)
- new net DDR_DQ3_B: U1.U2 (DQ3_b)
- new net DDR_DQ4_A: U1.F4 (DQ4_a)
- new net DDR_DQ4_B: U1.U4 (DQ4_b)
- new net DDR_DQ5_A: U1.E4 (DQ5_a)
- new net DDR_DQ5_B: U1.V4 (DQ5_b)
- new net DDR_DQ6_A: U1.C4 (DQ6_a)
- new net DDR_DQ6_B: U1.Y4 (DQ6_b)
- new net DDR_DQ7_A: U1.B4 (DQ7_a)
- new net DDR_DQ7_B: U1.AA4 (DQ7_b)
- new net DDR_DQ8_A: U1.B11 (DQ8_a)
- new net DDR_DQ8_B: U1.AA11 (DQ8_b)
- new net DDR_DQ9_A: U1.C11 (DQ9_a)
- new net DDR_DQ9_B: U1.Y11 (DQ9_b)
- new net DDR_DQS0N_A: U1.E3 (DQS0_c_a)
- new net DDR_DQS0N_B: U1.V3 (DQS0_c_b)
- new net DDR_DQS0P_A: U1.D3 (DQS0_t_a)
- new net DDR_DQS0P_B: U1.W3 (DQS0_t_b)
- new net DDR_DQS1N_A: U1.E10 (DQS1_c_a)
- new net DDR_DQS1N_B: U1.V10 (DQS1_c_b)
- new net DDR_DQS1P_A: U1.D10 (DQS1_t_a)
- new net DDR_DQS1P_B: U1.W10 (DQS1_t_b)
- new net DDR_ZQ0: R1.1, U1.A5 (ZQ0)
- new net DDR_ZQ1: R2.1, U1.A8 (ZQ1)
- new net GND: C1.2, C10.2, C11.2, C12.2, C13.2, C14.2, C15.2, C2.2, C3.2, C4.2, C5.2, C6.2, C7.2, C8.2, C9.2, R1.2, R2.2, U1.A10 (VSS), U1.A3 (VSS), U1.AB10 (VSS), U1.AB3 (VSS), U1.AB5 (VSS), U1.AB8 (VSS), U1.C1 (VSS), U1.C12 (VSS), U1.C5 (VSS), U1.C8 (VSS), U1.D11 (VSS), U1.D2 (VSS), U1.D4 (VSS), U1.D9 (VSS), U1.E1 (VSS), U1.E12 (VSS), U1.E5 (VSS), U1.E8 (VSS), U1.G1 (VSS), U1.G10 (VSS), U1.G12 (VSS), U1.G3 (VSS), U1.G5 (VSS), U1.G8 (VSS), U1.J1 (VSS), U1.J10 (VSS), U1.J12 (VSS), U1.J3 (VSS), U1.K11 (VSS), U1.K2 (VSS), U1.K4 (VSS), U1.K9 (VSS), U1.N11 (VSS), U1.N2 (VSS), U1.N4 (VSS), U1.N9 (VSS), U1.P1 (VSS), U1.P10 (VSS), U1.P12 (VSS), U1.P3 (VSS), U1.T1 (VSS), U1.T10 (VSS), U1.T12 (VSS), U1.T3 (VSS), U1.T5 (VSS), U1.T8 (VSS), U1.V1 (VSS), U1.V12 (VSS), U1.V5 (VSS), U1.V8 (VSS), U1.W11 (VSS), U1.W2 (VSS), U1.W4 (VSS), U1.W9 (VSS), U1.Y1 (VSS), U1.Y12 (VSS), U1.Y5 (VSS), U1.Y8 (VSS)
- new net LPDDR4_CA0_A: U1.H2 (CA0_a)
- new net LPDDR4_CA0_B: U1.R2 (CA0_b)
- new net LPDDR4_CA1_A: U1.J2 (CA1_a)
- new net LPDDR4_CA1_B: U1.P2 (CA1_b)
- new net LPDDR4_CA2_A: U1.H9 (CA2_a)
- new net LPDDR4_CA2_B: U1.R9 (CA2_b)
- new net LPDDR4_CA3_A: U1.H10 (CA3_a)
- new net LPDDR4_CA3_B: U1.R10 (CA3_b)
- new net LPDDR4_CA4_A: U1.H11 (CA4_a)
- new net LPDDR4_CA4_B: U1.R11 (CA4_b)
- new net LPDDR4_CA5_A: U1.J11 (CA5_a)
- new net LPDDR4_CA5_B: U1.P11 (CA5_b)
- new net LPDDR4_CKE0_A: U1.J4 (CKE0_a)
- new net LPDDR4_CKE0_B: U1.P4 (CKE0_b)
- new net LPDDR4_CKE1_A: U1.J5 (CKE1_a)
- new net LPDDR4_CKE1_B: U1.P5 (CKE1_b)
- new net LPDDR4_CK_C_A: U1.J9 (CK_c_a)
- new net LPDDR4_CK_C_B: U1.P9 (CK_c_b)
- new net LPDDR4_CK_T_A: U1.J8 (CK_t_a)
- new net LPDDR4_CK_T_B: U1.P8 (CK_t_b)
- new net LPDDR4_CS0_A: U1.H4 (CS0_a)
- new net LPDDR4_CS0_B: U1.R4 (CS0_b)
- new net LPDDR4_CS1_A: U1.H3 (CS1_a)
- new net LPDDR4_CS1_B: U1.R3 (CS1_b)
- new net LPDDR4_ODT_CA_A: U1.G2 (ODT_CA_a1)/2))
- new net LPDDR4_ODT_CA_B: U1.T2 (ODT_CA_b1)/2))
- new net LPDDR4_RESET_N: U1.T11 (RESET_n)
- new net VDD1_DDR: C1.1, C2.1, C3.1, C4.1, C5.1, U1.F1 (VDD1), U1.F12 (VDD1), U1.G4 (VDD1), U1.G9 (VDD1), U1.T4 (VDD1), U1.T9 (VDD1), U1.U1 (VDD1), U1.U12 (VDD1)
- new net VDD2_DDR: C10.1, C6.1, C7.1, C8.1, C9.1, U1.A4 (VDD2), U1.A9 (VDD2), U1.AB4 (VDD2), U1.AB9 (VDD2), U1.F5 (VDD2), U1.F8 (VDD2), U1.H1 (VDD2), U1.H12 (VDD2), U1.H5 (VDD2), U1.H8 (VDD2), U1.K1 (VDD2), U1.K10 (VDD2), U1.K12 (VDD2), U1.K3 (VDD2), U1.N1 (VDD2), U1.N10 (VDD2), U1.N12 (VDD2), U1.N3 (VDD2), U1.R1 (VDD2), U1.R12 (VDD2), U1.R5 (VDD2), U1.R8 (VDD2), U1.U5 (VDD2), U1.U8 (VDD2)
- new net VDDQ_DDR: C11.1, C12.1, C13.1, C14.1, C15.1, U1.AA10 (VDDQ), U1.AA3 (VDDQ), U1.AA5 (VDDQ), U1.AA8 (VDDQ), U1.B10 (VDDQ), U1.B3 (VDDQ), U1.B5 (VDDQ), U1.B8 (VDDQ), U1.D1 (VDDQ), U1.D12 (VDDQ), U1.D5 (VDDQ), U1.D8 (VDDQ), U1.F10 (VDDQ), U1.F3 (VDDQ), U1.U10 (VDDQ), U1.U3 (VDDQ), U1.W1 (VDDQ), U1.W12 (VDDQ), U1.W5 (VDDQ), U1.W8 (VDDQ)
- no-connect marks 0 -> 17

Commit message: display sheet
Other:
- title: (none) -> LPDDR4X Memory
Changed lines of the file:
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@@
 	(generator_version "10.0")
 	(paper "A3")
+	(title_block
+		(title "LPDDR4X Memory")
+	)
 					(number "T2"
 						(effects
