File: connectivity.kicad_sch (KiCad schematic)
At the start: 0 parts

Commit message: GPIO and root sheet
Parts:
- added C1, C2: 15pF, symbol Device:C
- added C59, C62: 100nF, symbol Device:C
- added C60: 4.7uF, symbol Device:C
- added C61, C63, C64: 10uF, symbol Device:C
- added J1: U.FL, symbol Connector:Conn_Coaxial
- added U1: AP6256, AP6256:QFN-44_L12.0-W12.0-P0.90-TL_AP6256, symbol AP6256:AP6256
- added Y1: 37.4MHz, symbol Device:Crystal
Connections:
- new net: C2.1, U1.11 (XTAL_OUT), Y1.1
- new net: C1.1, U1.10 (XTAL_IN), Y1.2
- new net: C60.2, U1.21 (VIN_LDO_OUT)
- new net: J1.1 (In), U1.2 (WL_BT_ANT)
- new net +1V8: C59.2, C63.2, U1.22 (VDDIO), U1.29 (SDIO_VSEL)
- new net +3V3: C61.2, C62.2, C64.2, U1.23 (VIN_LDO), U1.9 (VBAT)
- new net BT_HOST_WAKE: U1.7 (BT_HOST_WAKE)
- new net BT_REG_ON: U1.34 (BT_REG_ON)
- new net BT_UART_CTS: U1.44 (UART_CTS_N)
- new net BT_UART_RTS: U1.41 (UAR_RTS_N)
- new net BT_WAKE: U1.6 (BT_WAKE)
- new net GND: C1.2, C2.2, C59.1, C60.1, C61.1, C62.1, C63.1, C64.1, J1.2 (Ext), U1.1 (GND), U1.20 (GND), U1.3 (GND), U1.31 (GND), U1.33 (GND), U1.36 (GND)
- new net SDMMC1_CLK: U1.17 (SDIO_DATA_CLK)
- new net SDMMC1_CMD: U1.16 (SDIO_DATA_CMD)
- new net SDMMC1_D0: U1.18 (SDIO_DATA_0)
- new net SDMMC1_D1: U1.19 (SDIO_DATA_1)
- new net SDMMC1_D2: U1.14 (SDIO_DATA_2)
- new net SDMMC1_D3: U1.15 (SDIO_DATA_3)
- new net UART0_RX: U1.42 (UART_TXD)
- new net UART0_TX: U1.43 (UART_RXD)
- new net WIFI_CLK32K: U1.24 (LPO)
- new net WIFI_HOST_WAKE: U1.13 (WL_HOST_WAKE)
- new net WIFI_REG_ON: U1.12 (WL_REG_ON)
- no-connect marks 0 -> 17
Other:
- title: (none) -> WiFi/BLE

Commit message: root sheet changes
Parts:
- renumbered C1 to C104, C2 to C105, C63 to C106, C59 to C107, C64 to C108, C61 to C109, C62 to C110, C60 to C111, J1 to J5, U1 to U20, Y1 to Y5
Changed lines of the file:
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@@
 		(in_pos_files yes)
 		(dnp no)
-		(property "Reference" "#PWR094"
+		(property "Reference" "#PWR0183"
 			(at 104.14 81.28 0)
 			(hide yes)
@@
 			(project ""
 				(path "/6ade62f6-9cb2-4783-8048-f18138ca0ff8/b6eecf94-54f5-423d-adc8-5638173391e3"
-					(reference "#PWR094")
+					(reference "#PWR0183")
 					(unit 1)
 				)
@@
 		(in_pos_files yes)
 		(dnp no)
-		(property "Reference" "#PWR0103"
+		(property "Reference" "#PWR0192"
 			(at 194.31 111.76 0)
 			(hide yes)
@@
 			(project ""
 				(path "/6ade62f6-9cb2-4783-8048-f18138ca0ff8/b6eecf94-54f5-423d-adc8-5638173391e3"
-					(reference "#PWR0103")
+					(reference "#PWR0192")
 					(unit 1)
 				)
@@
 		(in_pos_files yes)
 		(dnp no)
-		(property "Reference" "#PWR096"
+		(property "Reference" "#PWR0180"
 			(at 100.33 115.57 0)
 			(hide yes)
@@
 			(project ""
 				(path "/6ade62f6-9cb2-4783-8048-f18138ca0ff8/b6eecf94-54f5-423d-adc8-5638173391e3"
-					(reference "#PWR096")
+					(reference "#PWR0180")
 					(unit 1)
 				)
@@
 		(in_pos_files yes)
 		(dnp no)
-		(property "Reference" "C63"
+		(property "Reference" "C106"
 			(at 109.22 114.935 0)
 			(show_name no)
@@
 			(project ""
 				(path "/6ade62f6-9cb2-4783-8048-f18138ca0ff8/b6eecf94-54f5-423d-adc8-5638173391e3"
-					(reference "C63")
+					(reference "C106")
 					(unit 1)
 				)
@@
 		(in_pos_files yes)
 		(dnp no)
-		(property "Reference" "#PWR2"
+		(property "Reference" "#PWR0178"
 			(at 93.98 96.52 0)
 			(hide yes)
@@
 			(project ""
 				(path "/6ade62f6-9cb2-4783-8048-f18138ca0ff8/b6eecf94-54f5-423d-adc8-5638173391e3"
-					(reference "#PWR2")
+					(reference "#PWR0178")
 					(unit 1)
 				)
@@
 		(in_pos_files yes)
 		(dnp no)
-		(property "Reference" "#PWR0102"
+		(property "Reference" "#PWR0191"
 			(at 194.31 106.68 0)
 			(hide yes)
@@
 			(project ""
 				(path "/6ade62f6-9cb2-4783-8048-f18138ca0ff8/b6eecf94-54f5-423d-adc8-5638173391e3"
-					(reference "#PWR0102")
+					(reference "#PWR0191")
 					(unit 1)
 				)
@@
 		(in_pos_files yes)
 		(dnp no)
-		(property "Reference" "#PWR092"
+		(property "Reference" "#PWR0181"
 			(at 100.33 123.19 0)
 			(hide yes)
@@
 			(project ""
 				(path "/6ade62f6-9cb2-4783-8048-f18138ca0ff8/b6eecf94-54f5-423d-adc8-5638173391e3"
-					(reference "#PWR092")
+					(reference "#PWR0181")
 					(unit 1)
 				)
@@
 		(in_pos_files yes)
 		(dnp no)
-		(property "Reference" "#PWR1"
+		(property "Reference" "#PWR0185"
 			(at 115.57 59.69 0)
 			(hide yes)
@@
 			(project ""
 				(path "/6ade62f6-9cb2-4783-8048-f18138ca0ff8/b6eecf94-54f5-423d-adc8-5638173391e3"
-					(reference "#PWR1")
+					(reference "#PWR0185")
 					(unit 1)
 				)
@@
 		(in_pos_files yes)
 		(dnp no)
-		(property "Reference" "#PWR099"
+		(property "Reference" "#PWR0188"
 			(at 130.81 74.93 0)
 			(hide yes)
@@
 			(project ""
 				(path "/6ade62f6-9cb2-4783-8048-f18138ca0ff8/b6eecf94-54f5-423d-adc8-5638173391e3"
-					(reference "#PWR099")
+					(reference "#PWR0188")
 					(unit 1)
 				)
@@
 		(in_pos_files yes)
 		(dnp no)
-		(property "Reference" "#PWR0100"
+		(property "Reference" "#PWR0189"
 			(at 130.81 118.11 0)
 			(hide yes)
@@
 			(project ""
 				(path "/6ade62f6-9cb2-4783-8048-f18138ca0ff8/b6eecf94-54f5-423d-adc8-5638173391e3"
-					(reference "#PWR0100")
+					(reference "#PWR0189")
 					(unit 1)
 				)
@@
 		(in_pos_files yes)
 		(dnp no)
-		(property "Reference" "C59"
+		(property "Reference" "C107"
 			(at 109.22 122.555 0)
 			(show_name no)
@@
 			(project ""
 				(path "/6ade62f6-9cb2-4783-8048-f18138ca0ff8/b6eecf94-54f5-423d-adc8-5638173391e3"
-					(reference "C59")
+					(reference "C107")
 					(unit 1)
 				)
@@
 		(in_pos_files yes)
 		(dnp no)
-		(property "Reference" "#PWR3"
+		(property "Reference" "#PWR0179"
 			(at 93.98 104.14 0)
 			(hide yes)
@@
 			(project ""
 				(path "/6ade62f6-9cb2-4783-8048-f18138ca0ff8/b6eecf94-54f5-423d-adc8-5638173391e3"
-					(reference "#PWR3")
+					(reference "#PWR0179")
 					(unit 1)
 				)
@@
 		(in_pos_files yes)
 		(dnp no)
-		(property "Reference" "#PWR097"
+		(property "Reference" "#PWR0182"
 			(at 100.33 130.81 0)
 			(hide yes)
@@
 			(project ""
 				(path "/6ade62f6-9cb2-4783-8048-f18138ca0ff8/b6eecf94-54f5-423d-adc8-5638173391e3"
-					(reference "#PWR097")
+					(reference "#PWR0182")
 					(unit 1)
 				)
@@
 		(in_pos_files yes)
 		(dnp no)
-		(property "Reference" "C62"
+		(property "Reference" "C110"
 			(at 113.03 86.995 0)
 			(show_name no)
@@
 			(project ""
 				(path "/6ade62f6-9cb2-4783-8048-f18138ca0ff8/b6eecf94-54f5-423d-adc8-5638173391e3"
-					(reference "C62")
+					(reference "C110")
 					(unit 1)
 				)
@@
 		(in_pos_files yes)
 		(dnp no)
-		(property "Reference" "Y1"
+		(property "Reference" "Y5"
 			(at 107.95 100.33 0)
 			(show_name no)
@@
 			(project ""
 				(path "/6ade62f6-9cb2-4783-8048-f18138ca0ff8/b6eecf94-54f5-423d-adc8-5638173391e3"
-					(reference "Y1")
+					(reference "Y5")
 					(unit 1)
 				)
@@
 		(in_pos_files yes)
 		(dnp no)
-		(property "Reference" "#PWR0104"
+		(property "Reference" "#PWR0193"
 			(at 184.15 116.84 0)
 			(hide yes)
@@
 			(project ""
 				(path "/6ade62f6-9cb2-4783-8048-f18138ca0ff8/b6eecf94-54f5-423d-adc8-5638173391e3"
-					(reference "#PWR0104")
+					(reference "#PWR0193")
 					(unit 1)
 				)
@@
 		(in_pos_files yes)
 		(dnp no)
-		(property "Reference" "C60"
+		(property "Reference" "C111"
 			(at 123.19 120.015 0)
 			(show_name no)
@@
 			(project ""
 				(path "/6ade62f6-9cb2-4783-8048-f18138ca0ff8/b6eecf94-54f5-423d-adc8-5638173391e3"
-					(reference "C60")
+					(reference "C111")
 					(unit 1)
 				)
@@
 		(in_pos_files yes)
 		(dnp no)
-		(property "Reference" "#PWR093"
+		(property "Reference" "#PWR0186"
 			(at 119.38 111.76 0)
 			(hide yes)
@@
 			(project ""
 				(path "/6ade62f6-9cb2-4783-8048-f18138ca0ff8/b6eecf94-54f5-423d-adc8-5638173391e3"
-					(reference "#PWR093")
+					(reference "#PWR0186")
 					(unit 1)
 				)
@@
 		(in_pos_files yes)
 		(dnp no)
-		(property "Reference" "U1"
+		(property "Reference" "U20"
 			(at 162.56 64.77 0)
 			(show_name no)
@@
 			(project ""
 				(path "/6ade62f6-9cb2-4783-8048-f18138ca0ff8/b6eecf94-54f5-423d-adc8-5638173391e3"
-					(reference "U1")
+					(reference "U20")
 					(unit 1)
 				)
@@
 		(in_pos_files yes)
 		(dnp no)
-		(property "Reference" "C2"
+		(property "Reference" "C105"
 			(at 106.68 102.362 0)
 			(show_name no)
@@
 			(project ""
 				(path "/6ade62f6-9cb2-4783-8048-f18138ca0ff8/b6eecf94-54f5-423d-adc8-5638173391e3"
-					(reference "C2")
+					(reference "C105")
 					(unit 1)
 				)
@@
 		(in_pos_files yes)
 		(dnp no)
-		(property "Reference" "#PWR095"
+		(property "Reference" "#PWR0184"
 			(at 104.14 87.63 0)
 			(hide yes)
@@
 			(project ""
 				(path "/6ade62f6-9cb2-4783-8048-f18138ca0ff8/b6eecf94-54f5-423d-adc8-5638173391e3"
-					(reference "#PWR095")
+					(reference "#PWR0184")
 					(unit 1)
 				)
@@
 		(in_pos_files yes)
 		(dnp no)
-		(property "Reference" "C1"
+		(property "Reference" "C104"
 			(at 106.68 94.234 0)
 			(show_name no)
@@
 			(project ""
 				(path "/6ade62f6-9cb2-4783-8048-f18138ca0ff8/b6eecf94-54f5-423d-adc8-5638173391e3"
-					(reference "C1")
+					(reference "C104")
 					(unit 1)
 				)
@@
 		(in_pos_files yes)
 		(dnp no)
-		(property "Reference" "C61"
+		(property "Reference" "C109"
 			(at 113.03 80.645 0)
 			(show_name no)
@@
 			(project ""
 				(path "/6ade62f6-9cb2-4783-8048-f18138ca0ff8/b6eecf94-54f5-423d-adc8-5638173391e3"
-					(reference "C61")
+					(reference "C109")
 					(unit 1)
 				)
@@
 		(in_pos_files yes)
 		(dnp no)
-		(property "Reference" "#PWR0101"
+		(property "Reference" "#PWR0190"
 			(at 194.31 99.06 0)
 			(hide yes)
@@
 			(project ""
 				(path "/6ade62f6-9cb2-4783-8048-f18138ca0ff8/b6eecf94-54f5-423d-adc8-5638173391e3"
-					(reference "#PWR0101")
+					(reference "#PWR0190")
 					(unit 1)
 				)
@@
 		(in_pos_files yes)
 		(dnp no)
-		(property "Reference" "J1"
+		(property "Reference" "J5"
 			(at 115.316 75.438 0)
 			(show_name no)
@@
 			(project ""
 				(path "/6ade62f6-9cb2-4783-8048-f18138ca0ff8/b6eecf94-54f5-423d-adc8-5638173391e3"
-					(reference "J1")
+					(reference "J5")
 					(unit 1)
 				)
@@
 		(in_pos_files yes)
 		(dnp no)
-		(property "Reference" "#PWR098"
+		(property "Reference" "#PWR0187"
 			(at 130.81 69.85 0)
 			(hide yes)
@@
 			(project ""
 				(path "/6ade62f6-9cb2-4783-8048-f18138ca0ff8/b6eecf94-54f5-423d-adc8-5638173391e3"
-					(reference "#PWR098")
+					(reference "#PWR0187")
 					(unit 1)
 				)
@@
 		(in_pos_files yes)
 		(dnp no)
-		(property "Reference" "C64"
+		(property "Reference" "C108"
 			(at 109.22 130.175 0)
 			(show_name no)
@@
 			(project ""
 				(path "/6ade62f6-9cb2-4783-8048-f18138ca0ff8/b6eecf94-54f5-423d-adc8-5638173391e3"
-					(reference "C64")
-					(unit 1)
-				)
+					(reference "C108")
+					(unit 1)
+				)
