File: display.kicad_sch (KiCad schematic)
At the start: 0 parts

Commit message: display sheet
Parts:
- added C44, C49, C50, C51, C52, C53, C54, C55: 100nF, symbol Device:C
- added R4, R5: 10k, symbol Device:R
- added U2: LT8711HE, project:QFN-64-1EP_7.5x7.5mm_P0.5mm, symbol LT8711HE:LT8711HE
- added U3: IT6505, Package_QFP:LQFP-144_20x20mm_P0.5mm, symbol IT6505:IT6505
- added Y3, Y4: 25MHz, symbol Device:Crystal
Connections:
- new net: R5.2, U3.59 (REXT)
- new net: U3.68 (XTALOUT), Y4.2
- new net: U2.37 (XTAL_OUT), Y3.2
- new net: R4.2, U2.32 (REXT)
- new net: C44.2, U2.7 (VCOMT)
- new net CSCL_GPIO3: U2.51 (CSCL_GPIO3)
- new net DP1_AUX_N: U3.39 (TXAUXN)
- new net DP1_AUX_P: U3.40 (TXAUXP)
- new net DP1_HPD: U3.37 (HPD)
- new net DP1_TX0_N: U3.55 (TX0N)
- new net DP1_TX0_P: U3.56 (TX0P)
- new net DP1_TX1_N: U3.51 (TX1N)
- new net DP1_TX1_P: U3.52 (TX1P)
- new net DP1_TX2_N: U3.47 (TX2N)
- new net DP1_TX2_P: U3.48 (TX2P)
- new net DP1_TX3_N: U3.43 (TX3N)
- new net DP1_TX3_P: U3.44 (TX3P)
- new net EDP_TX_AUXN: U2.35 (DRX_AUX-)
- new net EDP_TX_AUXP: U2.36 (DRX_AUX+)
- new net EDP_TX_D0N: U2.21 (D0N)
- new net EDP_TX_D0P: U2.20 (D0P)
- new net EDP_TX_D1N: U2.24 (D1N)
- new net EDP_TX_D1P: U2.23 (D1P)
- new net EDP_TX_D2N: U2.27 (D2N)
- new net EDP_TX_D2P: U2.26 (D2P)
- new net EDP_TX_D3N: U2.30 (D3N)
- new net EDP_TX_D3P: U2.29 (D3P)
- new net GND: C44.1, C49.1, C50.1, C51.1, C52.1, C53.1, C54.1, C55.1, R4.1, R5.1, U2.65 (VSS), U3.107 (IOVSS), U3.11 (IOVSS), U3.124 (IOVSS), U3.141 (IOVSS), U3.34 (IOVSS), U3.38 (AGND), U3.42 (AGND), U3.45 (AGND), U3.49 (AGND), U3.53 (AGND), U3.57 (AGND), U3.60 (AGND), U3.62 (PGND1), U3.64 (PGND2), U3.66 (PGND0), U3.70 (PGND0), U3.77 (IOVSS), U3.92 (IOVSS)
- new net HDMI_CEC: U2.34 (CEC_GPIO6)
- new net HDMI_CLK_N: U2.3 (HTX_C-)
- new net HDMI_CLK_P: U2.4 (HTX_C+)
- new net HDMI_DDC_SCL: U2.59 (HTX_DSCL)
- new net HDMI_DDC_SDA: U2.58 (HTX_DSDA)
- new net HDMI_HPD: U2.57 (HTX_HPD)
- new net HDMI_TX0_N: U2.5 (HTX_D0-)
- new net HDMI_TX0_P: U2.6 (HTX_D0+)
- new net HDMI_TX1_N: U2.10 (HTX_D1-)
- new net HDMI_TX1_P: U2.11 (HTX_D1+)
- new net HDMI_TX2_N: U2.12 (HTX_D2-)
- new net HDMI_TX2_P: U2.13 (HTX_D2+)
- new net IT6505_INT: U3.75 (~{INT})
- new net IT6505_RST_N: U3.36 (~{SYSRSTN})
- new net IT6505_SCL: U3.73 (PCSCL)
- new net IT6505_SDA: U3.74 (PCSDA)
- new net IT6505_XTAL: U3.69 (XTALIN), Y4.1
- new net LCDC_D0: U3.120 (OD0)
- new net LCDC_D1: U3.119 (OD1)
- new net LCDC_D10: U3.110 (OD10)
- new net LCDC_D11: U3.109 (OD11)
- new net LCDC_D12: U3.105 (OD12)
- new net LCDC_D13: U3.104 (OD13)
- new net LCDC_D14: U3.103 (OD14)
- new net LCDC_D15: U3.102 (OD15)
- new net LCDC_D16: U3.101 (OD16)
- new net LCDC_D17: U3.100 (OD17)
- new net LCDC_D18: U3.99 (OD18)
- new net LCDC_D19: U3.98 (OD19)
- new net LCDC_D2: U3.118 (OD2)
- new net LCDC_D20: U3.97 (OD20)
- new net LCDC_D21: U3.96 (OD21)
- new net LCDC_D22: U3.95 (OD22)
- new net LCDC_D23: U3.94 (OD23)
- new net LCDC_D3: U3.117 (OD3)
- new net LCDC_D4: U3.116 (OD4)
- new net LCDC_D5: U3.115 (OD5)
- new net LCDC_D6: U3.114 (OD6)
- new net LCDC_D7: U3.113 (OD7)
- new net LCDC_D8: U3.112 (OD8)
- new net LCDC_D9: U3.111 (OD9)
- new net LCDC_DCLK: U3.123 (PCLK)
- new net LCDC_DEN: U3.121 (DE)
- new net LCDC_HSYNC: U3.125 (HSYNC)
- new net LCDC_VSYNC: U3.126 (VSYNC)
- new net LT8711_INT: U2.46 (INTIO_GPIO2)
- new net LT8711_RST_N: U2.45 (RST_N)
- new net LT8711_SDA: U2.50 (CSDA_GPIO4)
- new net LT8711_XTAL: U2.38 (XTAL_IN), Y3.1
- new net USB_C_HDMI_CC1: U2.2 (DCC1)
- new net USB_C_HDMI_CC2: U2.41 (UCC2)
- new net USB_C_HDMI_CC2B: U2.1 (DCC2)
- new net USB_C_HDMI_HPD: U2.42 (UCC1_RXHPD)
- new net USB_C_HDMI_USB0_DN: U2.17 (USB0_DN)
- new net USB_C_HDMI_USB0_DP: U2.18 (USB0_DP)
- new net USB_C_HDMI_USB1_DN: U2.15 (USB1_DN)
- new net USB_C_HDMI_USB1_DP: U2.16 (USB1_DP)
- new net USB_C_HDMI_USB2_DN: U2.62 (USB2_DN)
- new net USB_C_HDMI_USB2_DP: U2.63 (USB2_DP)
- new net VBUS_HDMI: U2.33 (DVBUS)
- new net VCC1V2_DISP: C50.2, C52.2, C54.2, C55.2, U2.14 (VCC12), U2.19 (VCC12D_RX), U2.22 (VCC12A_RX), U2.28 (VCC12A_PI), U2.31 (VCC12A_RXPLL), U2.40 (VCC12), U2.48 (VCC12), U2.61 (VCC12), U2.64 (VCC12A_APLL), U2.9 (VCC12D_TX), U3.106 (IVDD), U3.12 (IVDD), U3.122 (IVDD), U3.140 (IVDD), U3.35 (IVDD), U3.41 (AVCC), U3.46 (AVCC), U3.50 (AVCC), U3.54 (AVCC), U3.58 (AVCC), U3.61 (PVCC1), U3.63 (PVCC2), U3.65 (PVCC0), U3.76 (IVDD), U3.91 (IVDD)
- new net VCC1V8_DISP: U3.67 (XVCC18)
- new net VCC3V3_DISP: C51.2, C53.2, U2.25 (VCC33A_RX), U2.43 (VCC33), U2.52 (VCC33), U2.8 (VCC33A_TX), U3.10 (OVDD), U3.108 (OVDD), U3.127 (OVDD), U3.33 (OVDD), U3.78 (OVDD), U3.93 (EMEM_VPP)
- new net VCC5V0: C49.2, U2.53 (VCC5)
- no-connect marks 0 -> 63

Commit message: USB Sheet
Other:
- title: (none) -> eDP and HDMI
Changed lines of the file:
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@@
 	(generator_version "10.0")
 	(paper "A3")
+	(title_block
+		(title "eDP and HDMI")
+	)
 	(junction
 		(at 110.49 228.6)

Commit message: root sheet changes
Parts:
- renumbered C52 to C59, C53 to C60, C54 to C61, C55 to C62, C50 to C63, C51 to C64, C49 to C65, C44 to C66, R5 to R3, U3 to U6, U2 to U7, Y4 to Y2
Changed lines of the file:
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@@
 		(in_pos_files yes)
 		(dnp no)
-		(property "Reference" "U3"
+		(property "Reference" "U6"
 			(at 137.668 228.092 0)
 			(show_name no)
@@
 			(project ""
 				(path "/6ade62f6-9cb2-4783-8048-f18138ca0ff8/93b2e130-37e3-4f18-9e2e-8e4bc19ffd57"
-					(reference "U3")
+					(reference "U6")
 					(unit 1)
 				)
@@
 		(in_pos_files yes)
 		(dnp no)
-		(property "Reference" "C49"
+		(property "Reference" "C65"
 			(at 353.06 142.875 0)
 			(show_name no)
@@
 			(project ""
 				(path "/6ade62f6-9cb2-4783-8048-f18138ca0ff8/93b2e130-37e3-4f18-9e2e-8e4bc19ffd57"
-					(reference "C49")
+					(reference "C65")
 					(unit 1)
 				)
@@
 		(in_pos_files yes)
 		(dnp no)
-		(property "Reference" "#PWR058"
+		(property "Reference" "#PWR064"
 			(at 113.03 46.99 0)
 			(hide yes)
@@
 			(project "test_board_20"
 				(path "/6ade62f6-9cb2-4783-8048-f18138ca0ff8/93b2e130-37e3-4f18-9e2e-8e4bc19ffd57"
-					(reference "#PWR058")
+					(reference "#PWR064")
 					(unit 1)
 				)
@@
 		(in_pos_files yes)
 		(dnp no)
-		(property "Reference" "#PWR055"
+		(property "Reference" "#PWR066"
 			(at 171.45 133.35 0)
 			(hide yes)
@@
 			(project "test_board_20"
 				(path "/6ade62f6-9cb2-4783-8048-f18138ca0ff8/93b2e130-37e3-4f18-9e2e-8e4bc19ffd57"
-					(reference "#PWR055")
+					(reference "#PWR066")
 					(unit 1)
 				)
@@
 		(in_pos_files yes)
 		(dnp no)
-		(property "Reference" "C51"
+		(property "Reference" "C64"
 			(at 353.06 132.715 0)
 			(show_name no)
@@
 			(project ""
 				(path "/6ade62f6-9cb2-4783-8048-f18138ca0ff8/93b2e130-37e3-4f18-9e2e-8e4bc19ffd57"
-					(reference "C51")
+					(reference "C64")
 					(unit 1)
 				)
@@
 		(in_pos_files yes)
 		(dnp no)
-		(property "Reference" "C55"
+		(property "Reference" "C62"
 			(at 126.365 55.88 0)
 			(show_name no)
@@
 			(project "test_board_20"
 				(path "/6ade62f6-9cb2-4783-8048-f18138ca0ff8/93b2e130-37e3-4f18-9e2e-8e4bc19ffd57"
-					(reference "C55")
+					(reference "C62")
 					(unit 1)
 				)
@@
 		(in_pos_files yes)
 		(dnp no)
-		(property "Reference" "#PWR052"
+		(property "Reference" "#PWR070"
 			(at 361.95 142.24 0)
 			(hide yes)
@@
 			(project ""
 				(path "/6ade62f6-9cb2-4783-8048-f18138ca0ff8/93b2e130-37e3-4f18-9e2e-8e4bc19ffd57"
-					(reference "#PWR052")
+					(reference "#PWR070")
 					(unit 1)
 				)
@@
 		(in_pos_files yes)
 		(dnp no)
-		(property "Reference" "Y4"
+		(property "Reference" "Y2"
 			(at 172.72 127 0)
 			(show_name no)
@@
 			(project "test_board_20"
 				(path "/6ade62f6-9cb2-4783-8048-f18138ca0ff8/93b2e130-37e3-4f18-9e2e-8e4bc19ffd57"
-					(reference "Y4")
+					(reference "Y2")
 					(unit 1)
 				)
@@
 		(in_pos_files yes)
 		(dnp no)
-		(property "Reference" "#PWR046"
+		(property "Reference" "#PWR067"
 			(at 349.25 147.32 0)
 			(hide yes)
@@
 			(project ""
 				(path "/6ade62f6-9cb2-4783-8048-f18138ca0ff8/93b2e130-37e3-4f18-9e2e-8e4bc19ffd57"
-					(reference "#PWR046")
+					(reference "#PWR067")
 					(unit 1)
 				)
@@
 		(in_pos_files yes)
 		(dnp no)
-		(property "Reference" "C53"
+		(property "Reference" "C60"
 			(at 100.965 55.88 0)
 			(show_name no)
@@
 			(project "test_board_20"
 				(path "/6ade62f6-9cb2-4783-8048-f18138ca0ff8/93b2e130-37e3-4f18-9e2e-8e4bc19ffd57"
-					(reference "C53")
+					(reference "C60")
 					(unit 1)
 				)
@@
 		(in_pos_files yes)
 		(dnp no)
-		(property "Reference" "C50"
+		(property "Reference" "C63"
 			(at 353.06 107.315 0)
 			(show_name no)
@@
 			(project ""
 				(path "/6ade62f6-9cb2-4783-8048-f18138ca0ff8/93b2e130-37e3-4f18-9e2e-8e4bc19ffd57"
-					(reference "C50")
+					(reference "C63")
 					(unit 1)
 				)
@@
 		(in_pos_files yes)
 		(dnp no)
-		(property "Reference" "R5"
+		(property "Reference" "R3"
 			(at 160.02 135.382 90)
 			(show_name no)
@@
 			(project "test_board_20"
 				(path "/6ade62f6-9cb2-4783-8048-f18138ca0ff8/93b2e130-37e3-4f18-9e2e-8e4bc19ffd57"
-					(reference "R5")
+					(reference "R3")
 					(unit 1)
 				)
@@
 		(in_pos_files yes)
 		(dnp no)
-		(property "Reference" "#PWR059"
+		(property "Reference" "#PWR065"
 			(at 125.73 46.99 0)
 			(hide yes)
@@
 			(project "test_board_20"
 				(path "/6ade62f6-9cb2-4783-8048-f18138ca0ff8/93b2e130-37e3-4f18-9e2e-8e4bc19ffd57"
-					(reference "#PWR059")
+					(reference "#PWR065")
 					(unit 1)
 				)
@@
 		(in_pos_files yes)
 		(dnp no)
-		(property "Reference" "#PWR054"
+		(property "Reference" "#PWR069"
 			(at 361.95 132.08 0)
 			(hide yes)
@@
 			(project ""
 				(path "/6ade62f6-9cb2-4783-8048-f18138ca0ff8/93b2e130-37e3-4f18-9e2e-8e4bc19ffd57"
-					(reference "#PWR054")
+					(reference "#PWR069")
 					(unit 1)
 				)
@@
 		(in_pos_files yes)
 		(dnp no)
-		(property "Reference" "#PWR057"
+		(property "Reference" "#PWR063"
 			(at 100.33 46.99 0)
 			(hide yes)
@@
 			(project "test_board_20"
 				(path "/6ade62f6-9cb2-4783-8048-f18138ca0ff8/93b2e130-37e3-4f18-9e2e-8e4bc19ffd57"
-					(reference "#PWR057")
+					(reference "#PWR063")
 					(unit 1)
 				)
@@
 		(in_pos_files yes)
 		(dnp no)
-		(property "Reference" "#PWR053"
+		(property "Reference" "#PWR068"
 			(at 361.95 106.68 0)
 			(hide yes)
@@
 			(project ""
 				(path "/6ade62f6-9cb2-4783-8048-f18138ca0ff8/93b2e130-37e3-4f18-9e2e-8e4bc19ffd57"
-					(reference "#PWR053")
+					(reference "#PWR068")
 					(unit 1)
 				)
@@
 		(in_pos_files yes)
 		(dnp no)
-		(property "Reference" "C52"
+		(property "Reference" "C59"
 			(at 83.185 55.88 0)
 			(show_name no)
@@
 			(project "test_board_20"
 				(path "/6ade62f6-9cb2-4783-8048-f18138ca0ff8/93b2e130-37e3-4f18-9e2e-8e4bc19ffd57"
-					(reference "C52")
+					(reference "C59")
 					(unit 1)
 				)
@@
 		(in_pos_files yes)
 		(dnp no)
-		(property "Reference" "C44"
+		(property "Reference" "C66"
 			(at 354.33 183.515 0)
 			(show_name no)
@@
 			(project ""
 				(path "/6ade62f6-9cb2-4783-8048-f18138ca0ff8/93b2e130-37e3-4f18-9e2e-8e4bc19ffd57"
-					(reference "C44")
+					(reference "C66")
 					(unit 1)
 				)
@@
 		(in_pos_files yes)
 		(dnp no)
-		(property "Reference" "#PWR056"
+		(property "Reference" "#PWR062"
 			(at 82.55 46.99 0)
 			(hide yes)
@@
 			(project "test_board_20"
 				(path "/6ade62f6-9cb2-4783-8048-f18138ca0ff8/93b2e130-37e3-4f18-9e2e-8e4bc19ffd57"
-					(reference "#PWR056")
+					(reference "#PWR062")
 					(unit 1)
 				)
@@
 		(in_pos_files yes)
 		(dnp no)
-		(property "Reference" "C54"
+		(property "Reference" "C61"
 			(at 113.665 55.88 0)
 			(show_name no)
@@
 			(project "test_board_20"
 				(path "/6ade62f6-9cb2-4783-8048-f18138ca0ff8/93b2e130-37e3-4f18-9e2e-8e4bc19ffd57"
-					(reference "C54")
+					(reference "C61")
 					(unit 1)
 				)
@@
 		(in_pos_files yes)
 		(dnp no)
-		(property "Reference" "#PWR047"
+		(property "Reference" "#PWR071"
 			(at 363.22 182.88 0)
 			(hide yes)
@@
 			(project ""
 				(path "/6ade62f6-9cb2-4783-8048-f18138ca0ff8/93b2e130-37e3-4f18-9e2e-8e4bc19ffd57"
-					(reference "#PWR047")
+					(reference "#PWR071")
 					(unit 1)
 				)
@@
 		(in_pos_files yes)
 		(dnp no)
-		(property "Reference" "U2"
+		(property "Reference" "U7"
 			(at 291.846 202.184 0)
 			(show_name no)
@@
 			(project ""
 				(path "/6ade62f6-9cb2-4783-8048-f18138ca0ff8/93b2e130-37e3-4f18-9e2e-8e4bc19ffd57"
-					(reference "U2")
-					(unit 1)
-				)
+					(reference "U7")
+					(unit 1)
+				)
