File: gpio_expansion.kicad_sch (KiCad schematic)
At the start: 0 parts

Commit message: GPIO and root sheet
Parts:
- added C65, C66: 100nF, symbol Device:C
- added D1: GREEN, symbol Device:LED
- added D2: RED, symbol Device:LED
- added J1: GPIO_Header, symbol Connector_Generic:Conn_02x20_Odd_Even
- added J2: Debug_UART, symbol Connector_Generic:Conn_01x03
- added J3: Micro_SD, symbol Connector:Micro_SD_Card_Det1
- added R1, R2: 1k, symbol Device:R
- added R7: 10k, symbol Device:R
- added SW1: RESET, symbol Switch:SW_Push
Connections:
- new net: D2.2 (A), R2.2
- new net: D1.2 (A), R1.2
- new net +3V3: C65.2, J1.1 (Pin_1), J1.17 (Pin_17), J3.4 (VDD), R1.1, R7.1
- new net +5V: J1.2 (Pin_2), J1.4 (Pin_4)
- new net GND: C65.1, C66.1, D1.1 (K), D2.1 (K), J1.14 (Pin_14), J1.20 (Pin_20), J1.25 (Pin_25), J1.30 (Pin_30), J1.34 (Pin_34), J1.39 (Pin_39), J1.6 (Pin_6), J1.9 (Pin_9), J2.3 (Pin_3), J3.10 (SHIELD), J3.6 (VSS), SW1.1
- new net GPIO0_A5: J1.27 (Pin_27)
- new net GPIO0_A6: J1.28 (Pin_28)
- new net GPIO2_D0: R2.1
- new net GPIO3_C0: J1.7 (Pin_7)
- new net GPIO3_C1: J1.11 (Pin_11)
- new net GPIO3_C2: J1.12 (Pin_12)
- new net GPIO3_C3: J1.13 (Pin_13)
- new net GPIO3_C4: J1.15 (Pin_15)
- new net GPIO3_C5: J1.16 (Pin_16)
- new net GPIO3_C6: J1.18 (Pin_18)
- new net GPIO3_C7: J1.22 (Pin_22)
- new net GPIO3_D2: J1.21 (Pin_21)
- new net GPIO3_D3: J1.19 (Pin_19)
- new net GPIO3_D4: J1.23 (Pin_23)
- new net GPIO3_D5: J1.24 (Pin_24)
- new net GPIO3_D6: J1.26 (Pin_26)
- new net GPIO3_D7: J1.29 (Pin_29)
- new net GPIO4_A0: J1.31 (Pin_31)
- new net GPIO4_A1: J1.32 (Pin_32)
- new net GPIO4_A2: J1.33 (Pin_33)
- new net GPIO4_A3: J1.35 (Pin_35)
- new net GPIO4_A4: J1.36 (Pin_36)
- new net GPIO4_A5: J1.38 (Pin_38)
- new net GPIO4_A6: J1.40 (Pin_40)
- new net I2C3_SCL: J1.5 (Pin_5)
- new net I2C3_SDA: J1.3 (Pin_3)
- new net SARADC_VIN0: J1.37 (Pin_37)
- new net SDMMC0_CLK: J3.5 (CLK)
- new net SDMMC0_CMD: J3.3 (CMD)
- new net SDMMC0_D0: J3.7 (DAT0)
- new net SDMMC0_D1: J3.8 (DAT1)
- new net SDMMC0_D2: J3.1 (DAT2)
- new net SDMMC0_D3: J3.2 (DAT3/CD)
- new net SDMMC0_DET: J3.9 (DET)
- new net UART2_RX: J1.10 (Pin_10), J2.2 (Pin_2)
- new net UART2_TX: J1.8 (Pin_8), J2.1 (Pin_1)
- new net nPOR: C66.2, R7.2, SW1.2

Commit message: root sheet changes
Parts:
- renumbered C65 to C112, C66 to C113, J1 to J6, J3 to J7, J2 to J8, R1 to R11, R2 to R12, R7 to R13
Changed lines of the file:
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@@
 		(in_pos_files yes)
 		(dnp no)
-		(property "Reference" "J2"
+		(property "Reference" "J8"
 			(at 243.84 64.77 0)
 			(show_name no)
@@
 			(project ""
 				(path "/6ade62f6-9cb2-4783-8048-f18138ca0ff8/6fa796a2-ee71-4756-9398-97fa015485e5"
-					(reference "J2")
+					(reference "J8")
 					(unit 1)
 				)
@@
 		(in_pos_files yes)
 		(dnp no)
-		(property "Reference" "#PWR0109"
+		(property "Reference" "#PWR0198"
 			(at 31.75 123.19 0)
 			(hide yes)
@@
 			(project ""
 				(path "/6ade62f6-9cb2-4783-8048-f18138ca0ff8/6fa796a2-ee71-4756-9398-97fa015485e5"
-					(reference "#PWR0109")
+					(reference "#PWR0198")
 					(unit 1)
 				)
@@
 		(in_pos_files yes)
 		(dnp no)
-		(property "Reference" "#PWR0117"
+		(property "Reference" "#PWR0212"
 			(at 231.14 72.39 0)
 			(hide yes)
@@
 			(project ""
 				(path "/6ade62f6-9cb2-4783-8048-f18138ca0ff8/6fa796a2-ee71-4756-9398-97fa015485e5"
-					(reference "#PWR0117")
+					(reference "#PWR0212")
 					(unit 1)
 				)
@@
 		(in_pos_files yes)
 		(dnp no)
-		(property "Reference" "J3"
+		(property "Reference" "J7"
 			(at 143.51 82.55 0)
 			(show_name no)
@@
 			(project ""
 				(path "/6ade62f6-9cb2-4783-8048-f18138ca0ff8/6fa796a2-ee71-4756-9398-97fa015485e5"
-					(reference "J3")
+					(reference "J7")
 					(unit 1)
 				)
@@
 		(in_pos_files yes)
 		(dnp no)
-		(property "Reference" "#PWR0115"
+		(property "Reference" "#PWR0204"
 			(at 83.82 110.49 0)
 			(hide yes)
@@
 			(project ""
 				(path "/6ade62f6-9cb2-4783-8048-f18138ca0ff8/6fa796a2-ee71-4756-9398-97fa015485e5"
-					(reference "#PWR0115")
+					(reference "#PWR0204")
 					(unit 1)
 				)
@@
 		(in_pos_files yes)
 		(dnp no)
-		(property "Reference" "R2"
+		(property "Reference" "R12"
 			(at 189.992 91.44 90)
 			(show_name no)
@@
 			(project ""
 				(path "/6ade62f6-9cb2-4783-8048-f18138ca0ff8/6fa796a2-ee71-4756-9398-97fa015485e5"
-					(reference "R2")
+					(reference "R12")
 					(unit 1)
 				)
@@
 		(in_pos_files yes)
 		(dnp no)
-		(property "Reference" "#PWR0105"
+		(property "Reference" "#PWR0194"
 			(at 41.91 74.93 0)
 			(hide yes)
@@
 			(project ""
 				(path "/6ade62f6-9cb2-4783-8048-f18138ca0ff8/6fa796a2-ee71-4756-9398-97fa015485e5"
-					(reference "#PWR0105")
+					(reference "#PWR0194")
 					(unit 1)
 				)
@@
 		(in_pos_files yes)
 		(dnp no)
-		(property "Reference" "#PWR0118"
+		(property "Reference" "#PWR0208"
 			(at 128.27 44.45 0)
 			(hide yes)
@@
 			(project ""
 				(path "/6ade62f6-9cb2-4783-8048-f18138ca0ff8/6fa796a2-ee71-4756-9398-97fa015485e5"
-					(reference "#PWR0118")
+					(reference "#PWR0208")
 					(unit 1)
 				)
@@
 		(in_pos_files yes)
 		(dnp no)
-		(property "Reference" "#PWR3"
+		(property "Reference" "#PWR0211"
 			(at 187.96 115.57 0)
 			(hide yes)
@@
 			(project ""
 				(path "/6ade62f6-9cb2-4783-8048-f18138ca0ff8/6fa796a2-ee71-4756-9398-97fa015485e5"
-					(reference "#PWR3")
+					(reference "#PWR0211")
 					(unit 1)
 				)
@@
 		(in_pos_files yes)
 		(dnp no)
-		(property "Reference" "R1"
+		(property "Reference" "R11"
 			(at 181.102 91.44 90)
 			(show_name no)
@@
 			(project ""
 				(path "/6ade62f6-9cb2-4783-8048-f18138ca0ff8/6fa796a2-ee71-4756-9398-97fa015485e5"
-					(reference "R1")
+					(reference "R11")
 					(unit 1)
 				)
@@
 		(in_pos_files yes)
 		(dnp no)
-		(property "Reference" "#PWR0119"
+		(property "Reference" "#PWR0207"
 			(at 123.19 50.8 0)
 			(hide yes)
@@
 			(project ""
 				(path "/6ade62f6-9cb2-4783-8048-f18138ca0ff8/6fa796a2-ee71-4756-9398-97fa015485e5"
-					(reference "#PWR0119")
+					(reference "#PWR0207")
 					(unit 1)
 				)
@@
 		(in_pos_files yes)
 		(dnp no)
-		(property "Reference" "#PWR0114"
+		(property "Reference" "#PWR0203"
 			(at 83.82 97.79 0)
 			(hide yes)
@@
 			(project ""
 				(path "/6ade62f6-9cb2-4783-8048-f18138ca0ff8/6fa796a2-ee71-4756-9398-97fa015485e5"
-					(reference "#PWR0114")
+					(reference "#PWR0203")
 					(unit 1)
 				)
@@
 		(in_pos_files yes)
 		(dnp no)
-		(property "Reference" "#PWR0116"
+		(property "Reference" "#PWR0205"
 			(at 83.82 115.57 0)
 			(hide yes)
@@
 			(project ""
 				(path "/6ade62f6-9cb2-4783-8048-f18138ca0ff8/6fa796a2-ee71-4756-9398-97fa015485e5"
-					(reference "#PWR0116")
+					(reference "#PWR0205")
 					(unit 1)
 				)
@@
 		(in_pos_files yes)
 		(dnp no)
-		(property "Reference" "#PWR0106"
+		(property "Reference" "#PWR0195"
 			(at 31.75 85.09 0)
 			(hide yes)
@@
 			(project ""
 				(path "/6ade62f6-9cb2-4783-8048-f18138ca0ff8/6fa796a2-ee71-4756-9398-97fa015485e5"
-					(reference "#PWR0106")
+					(reference "#PWR0195")
 					(unit 1)
 				)
@@
 		(in_pos_files yes)
 		(dnp no)
-		(property "Reference" "#PWR0110"
+		(property "Reference" "#PWR0199"
 			(at 73.66 69.85 0)
 			(hide yes)
@@
 			(project ""
 				(path "/6ade62f6-9cb2-4783-8048-f18138ca0ff8/6fa796a2-ee71-4756-9398-97fa015485e5"
-					(reference "#PWR0110")
+					(reference "#PWR0199")
 					(unit 1)
 				)
@@
 		(in_pos_files yes)
 		(dnp no)
-		(property "Reference" "#PWR2"
+		(property "Reference" "#PWR0210"
 			(at 179.07 115.57 0)
 			(hide yes)
@@
 			(project ""
 				(path "/6ade62f6-9cb2-4783-8048-f18138ca0ff8/6fa796a2-ee71-4756-9398-97fa015485e5"
-					(reference "#PWR2")
+					(reference "#PWR0210")
 					(unit 1)
 				)
@@
 		(in_pos_files yes)
 		(dnp no)
-		(property "Reference" "#PWR1"
+		(property "Reference" "#PWR0209"
 			(at 179.07 90.17 0)
 			(hide yes)
@@
 			(project ""
 				(path "/6ade62f6-9cb2-4783-8048-f18138ca0ff8/6fa796a2-ee71-4756-9398-97fa015485e5"
-					(reference "#PWR1")
+					(reference "#PWR0209")
 					(unit 1)
 				)
@@
 		(in_pos_files yes)
 		(dnp no)
-		(property "Reference" "#PWR0108"
+		(property "Reference" "#PWR0197"
 			(at 31.75 105.41 0)
 			(hide yes)
@@
 			(project ""
 				(path "/6ade62f6-9cb2-4783-8048-f18138ca0ff8/6fa796a2-ee71-4756-9398-97fa015485e5"
-					(reference "#PWR0108")
+					(reference "#PWR0197")
 					(unit 1)
 				)
@@
 		(in_pos_files yes)
 		(dnp no)
-		(property "Reference" "#PWR0113"
+		(property "Reference" "#PWR0202"
 			(at 83.82 90.17 0)
 			(hide yes)
@@
 			(project ""
 				(path "/6ade62f6-9cb2-4783-8048-f18138ca0ff8/6fa796a2-ee71-4756-9398-97fa015485e5"
-					(reference "#PWR0113")
+					(reference "#PWR0202")
 					(unit 1)
 				)
@@
 		(in_pos_files yes)
 		(dnp no)
-		(property "Reference" "#PWR0111"
+		(property "Reference" "#PWR0200"
 			(at 73.66 74.93 0)
 			(hide yes)
@@
 			(project ""
 				(path "/6ade62f6-9cb2-4783-8048-f18138ca0ff8/6fa796a2-ee71-4756-9398-97fa015485e5"
-					(reference "#PWR0111")
+					(reference "#PWR0200")
 					(unit 1)
 				)
@@
 		(in_pos_files yes)
 		(dnp no)
-		(property "Reference" "C66"
+		(property "Reference" "C113"
 			(at 247.015 96.52 0)
 			(show_name no)
@@
 			(project ""
 				(path "/6ade62f6-9cb2-4783-8048-f18138ca0ff8/6fa796a2-ee71-4756-9398-97fa015485e5"
-					(reference "C66")
+					(reference "C113")
 					(unit 1)
 				)
@@
 		(in_pos_files yes)
 		(dnp no)
-		(property "Reference" "#PWR0122"
+		(property "Reference" "#PWR0213"
 			(at 238.76 97.79 0)
 			(hide yes)
@@
 			(project ""
 				(path "/6ade62f6-9cb2-4783-8048-f18138ca0ff8/6fa796a2-ee71-4756-9398-97fa015485e5"
-					(reference "#PWR0122")
+					(reference "#PWR0213")
 					(unit 1)
 				)
@@
 		(in_pos_files yes)
 		(dnp no)
-		(property "Reference" "C65"
+		(property "Reference" "C112"
 			(at 128.905 53.34 0)
 			(show_name no)
@@
 			(project ""
 				(path "/6ade62f6-9cb2-4783-8048-f18138ca0ff8/6fa796a2-ee71-4756-9398-97fa015485e5"
-					(reference "C65")
+					(reference "C112")
 					(unit 1)
 				)
@@
 		(in_pos_files yes)
 		(dnp no)
-		(property "Reference" "#PWR0107"
+		(property "Reference" "#PWR0196"
 			(at 41.91 95.25 0)
 			(hide yes)
@@
 			(project ""
 				(path "/6ade62f6-9cb2-4783-8048-f18138ca0ff8/6fa796a2-ee71-4756-9398-97fa015485e5"
-					(reference "#PWR0107")
+					(reference "#PWR0196")
 					(unit 1)
 				)
@@
 		(in_pos_files yes)
 		(dnp no)
-		(property "Reference" "R7"
+		(property "Reference" "R13"
 			(at 240.792 99.06 90)
 			(show_name no)
@@
 			(project ""
 				(path "/6ade62f6-9cb2-4783-8048-f18138ca0ff8/6fa796a2-ee71-4756-9398-97fa015485e5"
-					(reference "R7")
+					(reference "R13")
 					(unit 1)
 				)
@@
 		(in_pos_files yes)
 		(dnp no)
-		(property "Reference" "J1"
+		(property "Reference" "J6"
 			(at 58.42 72.39 0)
 			(show_name no)
@@
 			(project ""
 				(path "/6ade62f6-9cb2-4783-8048-f18138ca0ff8/6fa796a2-ee71-4756-9398-97fa015485e5"
-					(reference "J1")
+					(reference "J6")
 					(unit 1)
 				)
@@
 		(in_pos_files yes)
 		(dnp no)
-		(property "Reference" "#PWR0123"
+		(property "Reference" "#PWR0215"
 			(at 246.38 87.63 0)
 			(hide yes)
@@
 			(project ""
 				(path "/6ade62f6-9cb2-4783-8048-f18138ca0ff8/6fa796a2-ee71-4756-9398-97fa015485e5"
-					(reference "#PWR0123")
+					(reference "#PWR0215")
 					(unit 1)
 				)
@@
 		(in_pos_files yes)
 		(dnp no)
-		(property "Reference" "#PWR0112"
+		(property "Reference" "#PWR0201"
 			(at 83.82 80.01 0)
 			(hide yes)
@@
 			(project ""
 				(path "/6ade62f6-9cb2-4783-8048-f18138ca0ff8/6fa796a2-ee71-4756-9398-97fa015485e5"
-					(reference "#PWR0112")
+					(reference "#PWR0201")
 					(unit 1)
 				)
@@
 		(in_pos_files yes)
 		(dnp no)
-		(property "Reference" "#PWR0121"
+		(property "Reference" "#PWR0214"
 			(at 238.76 127 0)
 			(hide yes)
@@
 			(project ""
 				(path "/6ade62f6-9cb2-4783-8048-f18138ca0ff8/6fa796a2-ee71-4756-9398-97fa015485e5"
-					(reference "#PWR0121")
+					(reference "#PWR0214")
 					(unit 1)
 				)
@@
 		(in_pos_files yes)
 		(dnp no)
-		(property "Reference" "#PWR0120"
+		(property "Reference" "#PWR0206"
 			(at 113.03 127 0)
 			(hide yes)
@@
 			(project ""
 				(path "/6ade62f6-9cb2-4783-8048-f18138ca0ff8/6fa796a2-ee71-4756-9398-97fa015485e5"
-					(reference "#PWR0120")
-					(unit 1)
-				)
+					(reference "#PWR0206")
+					(unit 1)
+				)
