File: lpddr4x.kicad_sch (KiCad schematic)
At the start: 18 parts, among them U13 K4UCE3Q4AB-MGCL

Commit message: GPIO and root sheet
Other:
- title: (none) -> LPDDR4X Memory
Changed lines of the file:
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@@
 	(generator_version "10.0")
 	(paper "A4" portrait)
+	(title_block
+		(title "LPDDR4X Memory")
+	)
 					(number "T2"
 						(effects

Commit message: root sheet changes
Parts:
- renumbered C67 to C37, C68 to C38, C69 to C39, C70 to C40, C71 to C41, C72 to C42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
