File: power_supply.kicad_sch (KiCad schematic)
At the start: 43 parts, among them U1 RK809-5, Y1 Crystal

Commit message: display sheet
Other:
- title: (none) -> PMIC
Changed lines of the file:
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@@
 	(generator_version "10.0")
 	(paper "A3")
+	(title_block
+		(title "PMIC")
+	)
 	(no_connect
 		(at 231.14 104.14)

Commit message: root sheet changes
Parts:
- renumbered C25 to C1, C4 to C10, C29 to C11, C16 to C12, C1 to C13, C30 to C14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
