File: storage.kicad_sch (KiCad schematic)
At the start: 0 parts

Commit message: display sheet
Parts:
- added C37, C38, C40, C41, C43: 100nF, symbol Device:C
- added C39, C42: 10uF, symbol Device:C
- added U1: KLMBG2JETD-B041, KLMBG2JETD-B041:FBGA-153_L13.0-W11.5-P0.50_KLMAG1JETD-B041, symbol KLMBG2JETD-B041:KLMBG2JETD-B041
- added U4: W25Q128JVS, Package_SO:SOIC-8_5.3x5.3mm_P1.27mm, symbol Memory_Flash:W25Q128JVS
Connections:
- new net EMMC_CLK: U1.M6 (CLK)
- new net EMMC_CMD: U1.M5 (CDM)
- new net EMMC_D0: U1.A3 (DAT0)
- new net EMMC_D1: U1.A4 (DAT1)
- new net EMMC_D2: U1.A5 (DAT2)
- new net EMMC_D3: U1.B2 (DAT3)
- new net EMMC_D4: U1.B3 (DAT4)
- new net EMMC_D5: U1.B4 (DAT5)
- new net EMMC_D6: U1.B5 (DAT6)
- new net EMMC_D7: U1.B6 (DAT7)
- new net EMMC_DATA_STROBE: U1.H5 (DATA-STROBE)
- new net EMMC_RSTN: U1.K5 (RSTN)
- new net GND: C37.1, C38.1, C39.1, C40.1, C41.1, C42.1, C43.1, U1.A6 (VSS), U1.C4 (VSS), U1.E7 (VSS), U1.G5 (VSS), U1.H10 (VSS), U1.J5 (VSS), U1.K8 (VSS), U1.N2 (VSS), U1.N5 (VSS), U1.P4 (VSS), U1.P6 (VSS), U4.4 (GND)
- new net SPI_FLASH_CLK: U4.6 (CLK)
- new net SPI_FLASH_CS: U4.1 (~{CS})
- new net SPI_FLASH_HOLD: U4.7 (~{HOLD}/~{RESET}/IO_{3})
- new net SPI_FLASH_MISO: U4.2 (DO/IO_{1})
- new net SPI_FLASH_MOSI: U4.5 (DI/IO_{0})
- new net SPI_FLASH_WP: U4.3 (~{WP}/IO_{2})
- new net VCC1V8_EMMC: C38.2, U1.C2 (VDDI)
- new net VCC3V3_EMMC: C39.2, C40.2, C41.2, C42.2, C43.2, U1.C6 (VDD), U1.E6 (VDDF), U1.F5 (VDDF), U1.J10 (VDDF), U1.K9 (VDDF), U1.M4 (VDD), U1.N4 (VDD), U1.P3 (VDD), U1.P5 (VDD)
- new net VCC3V3_SYS: C37.2, U4.8 (VCC)
- no-connect marks 0 -> 120
Other:
- title: (none) -> eMMC Storage

Commit message: root sheet changes
Parts:
- renumbered C38 to C52, C39 to C53, C40 to C54, C41 to C55, C43 to C56, C42 to C57, C37 to C58, U1 to U4, U4 to U5
Changed lines of the file:
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@@
 		(in_pos_files yes)
 		(dnp no)
-		(property "Reference" "C37"
+		(property "Reference" "C58"
 			(at 300.355 110.49 0)
 			(show_name no)
@@
 			(project ""
 				(path "/6ade62f6-9cb2-4783-8048-f18138ca0ff8/2988873c-a49d-4427-8b5f-52350d5f3ce7"
-					(reference "C37")
+					(reference "C58")
 					(unit 1)
 				)
@@
 		(in_pos_files yes)
 		(dnp no)
-		(property "Reference" "C40"
+		(property "Reference" "C54"
 			(at 73.66 86.995 0)
 			(show_name no)
@@
 			(project ""
 				(path "/6ade62f6-9cb2-4783-8048-f18138ca0ff8/2988873c-a49d-4427-8b5f-52350d5f3ce7"
-					(reference "C40")
+					(reference "C54")
 					(unit 1)
 				)
@@
 		(in_pos_files yes)
 		(dnp no)
-		(property "Reference" "#PWR042"
+		(property "Reference" "#PWR058"
 			(at 64.77 107.95 0)
 			(hide yes)
@@
 			(project ""
 				(path "/6ade62f6-9cb2-4783-8048-f18138ca0ff8/2988873c-a49d-4427-8b5f-52350d5f3ce7"
-					(reference "#PWR042")
+					(reference "#PWR058")
 					(unit 1)
 				)
@@
 		(in_pos_files yes)
 		(dnp no)
-		(property "Reference" "#PWR038"
+		(property "Reference" "#PWR061"
 			(at 299.72 101.6 0)
 			(hide yes)
@@
 			(project ""
 				(path "/6ade62f6-9cb2-4783-8048-f18138ca0ff8/2988873c-a49d-4427-8b5f-52350d5f3ce7"
-					(reference "#PWR038")
+					(reference "#PWR061")
 					(unit 1)
 				)
@@
 		(in_pos_files yes)
 		(dnp no)
-		(property "Reference" "U1"
+		(property "Reference" "U4"
 			(at 119.38 46.99 0)
 			(show_name no)
@@
 			(project ""
 				(path "/6ade62f6-9cb2-4783-8048-f18138ca0ff8/2988873c-a49d-4427-8b5f-52350d5f3ce7"
-					(reference "U1")
+					(reference "U4")
 					(unit 1)
 				)
@@
 		(in_pos_files yes)
 		(dnp no)
-		(property "Reference" "#PWR043"
+		(property "Reference" "#PWR060"
 			(at 64.77 130.81 0)
 			(hide yes)
@@
 			(project ""
 				(path "/6ade62f6-9cb2-4783-8048-f18138ca0ff8/2988873c-a49d-4427-8b5f-52350d5f3ce7"
-					(reference "#PWR043")
+					(reference "#PWR060")
 					(unit 1)
 				)
@@
 		(in_pos_files yes)
 		(dnp no)
-		(property "Reference" "#PWR040"
+		(property "Reference" "#PWR056"
 			(at 64.77 80.01 0)
 			(hide yes)
@@
 			(project ""
 				(path "/6ade62f6-9cb2-4783-8048-f18138ca0ff8/2988873c-a49d-4427-8b5f-52350d5f3ce7"
-					(reference "#PWR040")
+					(reference "#PWR056")
 					(unit 1)
 				)
@@
 		(in_pos_files yes)
 		(dnp no)
-		(property "Reference" "C38"
+		(property "Reference" "C52"
 			(at 73.66 74.295 0)
 			(show_name no)
@@
 			(project ""
 				(path "/6ade62f6-9cb2-4783-8048-f18138ca0ff8/2988873c-a49d-4427-8b5f-52350d5f3ce7"
-					(reference "C38")
+					(reference "C52")
 					(unit 1)
 				)
@@
 		(in_pos_files yes)
 		(dnp no)
-		(property "Reference" "C41"
+		(property "Reference" "C55"
 			(at 73.66 107.315 0)
 			(show_name no)
@@
 			(project ""
 				(path "/6ade62f6-9cb2-4783-8048-f18138ca0ff8/2988873c-a49d-4427-8b5f-52350d5f3ce7"
-					(reference "C41")
+					(reference "C55")
 					(unit 1)
 				)
@@
 		(in_pos_files yes)
 		(dnp no)
-		(property "Reference" "C39"
+		(property "Reference" "C53"
 			(at 73.66 79.375 0)
 			(show_name no)
@@
 			(project ""
 				(path "/6ade62f6-9cb2-4783-8048-f18138ca0ff8/2988873c-a49d-4427-8b5f-52350d5f3ce7"
-					(reference "C39")
+					(reference "C53")
 					(unit 1)
 				)
@@
 		(in_pos_files yes)
 		(dnp no)
-		(property "Reference" "#PWR044"
+		(property "Reference" "#PWR059"
 			(at 64.77 115.57 0)
 			(hide yes)
@@
 			(project ""
 				(path "/6ade62f6-9cb2-4783-8048-f18138ca0ff8/2988873c-a49d-4427-8b5f-52350d5f3ce7"
-					(reference "#PWR044")
+					(reference "#PWR059")
 					(unit 1)
 				)
@@
 		(in_pos_files yes)
 		(dnp no)
-		(property "Reference" "C43"
+		(property "Reference" "C56"
 			(at 73.66 114.935 0)
 			(show_name no)
@@
 			(project ""
 				(path "/6ade62f6-9cb2-4783-8048-f18138ca0ff8/2988873c-a49d-4427-8b5f-52350d5f3ce7"
-					(reference "C43")
+					(reference "C56")
 					(unit 1)
 				)
@@
 		(in_pos_files yes)
 		(dnp no)
-		(property "Reference" "#PWR041"
+		(property "Reference" "#PWR057"
 			(at 64.77 87.63 0)
 			(hide yes)
@@
 			(project ""
 				(path "/6ade62f6-9cb2-4783-8048-f18138ca0ff8/2988873c-a49d-4427-8b5f-52350d5f3ce7"
-					(reference "#PWR041")
+					(reference "#PWR057")
 					(unit 1)
 				)
@@
 		(dnp no)
 		(fields_autoplaced yes)
-		(property "Reference" "U4"
+		(property "Reference" "U5"
 			(at 311.15 135.8899 0)
 			(show_name no)
@@
 			(project ""
 				(path "/6ade62f6-9cb2-4783-8048-f18138ca0ff8/2988873c-a49d-4427-8b5f-52350d5f3ce7"
-					(reference "U4")
+					(reference "U5")
 					(unit 1)
 				)
@@
 		(in_pos_files yes)
 		(dnp no)
-		(property "Reference" "C42"
+		(property "Reference" "C57"
 			(at 73.66 130.175 0)
 			(show_name no)
@@
 			(project ""
 				(path "/6ade62f6-9cb2-4783-8048-f18138ca0ff8/2988873c-a49d-4427-8b5f-52350d5f3ce7"
-					(reference "C42")
+					(reference "C57")
 					(unit 1)
 				)
@@
 		(in_pos_files yes)
 		(dnp no)
-		(property "Reference" "#PWR039"
+		(property "Reference" "#PWR055"
 			(at 64.77 74.93 0)
 			(hide yes)
@@
 			(project ""
 				(path "/6ade62f6-9cb2-4783-8048-f18138ca0ff8/2988873c-a49d-4427-8b5f-52350d5f3ce7"
-					(reference "#PWR039")
+					(reference "#PWR055")
 					(unit 1)
 				)
