File: test_board_20.kicad_sch (KiCad schematic)
At the start: 0 parts

Commit message: PMIC sheet
Other:
- added sheet Connectivity (connectivity.kicad_sch)
- added sheet DDR Memory (ddr_memory.kicad_sch)
- added sheet Display (display.kicad_sch)
- added sheet GPIO and Expansion (gpio_expansion.kicad_sch)
- added sheet Power Supply (power_supply.kicad_sch)
- added sheet SoC (soc.kicad_sch)
- added sheet Storage (storage.kicad_sch)
- added sheet USB (usb.kicad_sch)

Commit message: soc board
Other:
- sheet Power Supply ports: added VCC_DDR, VDC, VDD_CPU, VDD_GPU, VDD_LOGIC, VDD_NPU; removed none
- sheet SoC ports: added CLK32K_IN, CLK32K_OUT1, DDR4_A0, DDR4_A1, DDR4_A10, DDR4_A11, DDR4_A12, DDR4_A13, DDR4_A14_WEn, DDR4_A15_CASn, DDR4_A16_RASn, DDR4_A2, DDR4_A3, DDR4_A4, DDR4_A5, DDR4_A6, DDR4_A7, DDR4_A8, DDR4_A9, DDR4_ACTn, DDR4_BA0, DDR4_BA1, DDR4_BG0, DDR4_BG1, DDR4_CKE, DDR4_CLKN, DDR4_CLKP, DDR4_CS0n, DDR4_CS1n, DDR4_ODT0, DDR4_ODT1, DDR4_RESETn, DDR_DM0_A, DDR_DM0_B, DDR_DM1_A, DDR_DM1_B, DDR_DQ0_A, DDR_DQ0_B, DDR_DQ10_A, DDR_DQ10_B, DDR_DQ11_A, DDR_DQ11_B, DDR_DQ12_A, DDR_DQ12_B, DDR_DQ13_A, DDR_DQ13_B, DDR_DQ14_A, DDR_DQ14_B, DDR_DQ15_A, DDR_DQ15_B, DDR_DQ1_A, DDR_DQ1_B, DDR_DQ2_A, DDR_DQ2_B, DDR_DQ3_A, DDR_DQ3_B, DDR_DQ4_A, DDR_DQ4_B, DDR_DQ5_A, DDR_DQ5_B, DDR_DQ6_A, DDR_DQ6_B, DDR_DQ7_A, DDR_DQ7_B, DDR_DQ8_A, DDR_DQ8_B, DDR_DQ9_A, DDR_DQ9_B, DDR_DQS0N_A, DDR_DQS0N_B, DDR_DQS0P_A, DDR_DQS0P_B, DDR_DQS1N_A, DDR_DQS1N_B, DDR_DQS1P_A, DDR_DQS1P_B, DDR_ECC_DM, DDR_ECC_DQ0, DDR_ECC_DQ1, DDR_ECC_DQ2, DDR_ECC_DQ3, DDR_ECC_DQ4, DDR_ECC_DQ5, DDR_ECC_DQ6, DDR_ECC_DQ7, DDR_ECC_DQS_N, DDR_ECC_DQS_P, DDR_RZQ, DDR_VREFOUT, EDP_HPDIN, EDP_TX_AUXN, EDP_TX_AUXP, EDP_TX_AVDD_0V9, EDP_TX_AVDD_1V8, EDP_TX_D0N, EDP_TX_D0P, EDP_TX_D1N, EDP_TX_D1P, EDP_TX_D2N, EDP_TX_D2P, EDP_TX_D3N, EDP_TX_D3P, EMMC_CLKOUT, EMMC_CMD, EMMC_D0, EMMC_D1, EMMC_D2, EMMC_D3, EMMC_D4, EMMC_D5, EMMC_D6, EMMC_D7, EMMC_DATA_STROBE, EMMC_RSTn, FLASH_VOL_SEL, FSPI_CLK, FSPI_CS0n, FSPI_D0, FSPI_D1, FSPI_D3, GMAC0_ETH_REFCLK, GMAC0_MCLKINOUT, GMAC0_MDC, GMAC0_MDIO, GMAC0_RXD0, GMAC0_RXD1, GMAC0_RXDV_CRS, GMAC0_RXER, GMAC0_TXD0, GMAC0_TXD1, GMAC0_TXEN, GPIO0_A3, GPIO0_A5, GPIO0_A6, GPIO0_B2, GPIO0_B4, GPIO0_B5, GPIO0_B6, GPIO0_B7, GPIO0_C2, GPIO0_C3, GPIO0_C4, GPIO0_C5, GPIO0_C6, GPIO0_C7, GPIO0_D3, GPIO0_D4, GPIO0_D5, GPIO0_D6, GPIO1_A2, GPIO1_A3, GPIO1_A4, GPIO1_A5, GPIO1_A6, GPIO1_A7, GPIO1_B0, GPIO1_B1, GPIO1_B2, GPIO1_B3, GPIO2_D0, GPIO2_D1, GPIO2_D2, GPIO2_D3, GPIO2_D4, GPIO2_D5, GPIO2_D6, GPIO2_D7, GPIO3_A0, GPIO3_A1, GPIO3_A2, GPIO3_A3, GPIO3_A4, GPIO3_A5, GPIO3_A6, GPIO3_A7, GPIO3_B0, GPIO3_B1, GPIO3_B2, GPIO3_B3, GPIO3_B4, GPIO3_B5, GPIO3_B6, GPIO3_B7, GPIO3_C0, GPIO3_C1, GPIO3_C2, GPIO3_C3, GPIO3_C4, GPIO3_C5, GPIO3_C6, GPIO3_C7, GPIO3_D0, GPIO3_D1, GPIO3_D2, GPIO3_D3, GPIO3_D4, GPIO3_D5, GPIO3_D6, GPIO3_D7, GPIO4_A0, GPIO4_A1, GPIO4_A2, GPIO4_A3, GPIO4_A4, GPIO4_A5, GPIO4_A6, GPIO4_A7, GPIO4_B0, GPIO4_B1, GPIO4_B2, GPIO4_B3, GPIO4_B4, GPIO4_B5, GPIO4_B6, GPIO4_B7, GPIO4_C0, GPIO4_C1, GPIO4_C2, GPIO4_C3, GPIO4_C5, GPIO4_C6, GPIO4_D2, HDMITX_CEC, HDMITX_SCL, HDMITX_SDA, HDMI_TX_AVDD_0V9, HDMI_TX_AVDD_1V8, HDMI_TX_CLKN, HDMI_TX_CLKP, HDMI_TX_D0N, HDMI_TX_D0P, HDMI_TX_D1N, HDMI_TX_D1P, HDMI_TX_D2N, HDMI_TX_D2P, HDMI_TX_HPDIN, HDMI_TX_REXT, I2C0_SCL, I2C1_SCL, I2C3_SCL, I2C3_SDA, MIPI_CSI_RX_AVDD_0V9, MIPI_CSI_RX_AVDD_1V8, MIPI_CSI_RX_CLK0N, MIPI_CSI_RX_CLK0P, MIPI_CSI_RX_CLK1N, MIPI_CSI_RX_CLK1P, MIPI_CSI_RX_D0N, MIPI_CSI_RX_D0P, MIPI_CSI_RX_D1N, MIPI_CSI_RX_D1P, MIPI_CSI_RX_D2N, MIPI_CSI_RX_D2P, MIPI_CSI_RX_D3N, MIPI_CSI_RX_D3P, MIPI_DSI_TX0_AVDD_0V9, MIPI_DSI_TX0_AVDD_1V8, MIPI_DSI_TX0_CLKN, MIPI_DSI_TX0_CLKP, MIPI_DSI_TX0_D0N, MIPI_DSI_TX0_D0P, MIPI_DSI_TX0_D1N, MIPI_DSI_TX0_D1P, MIPI_DSI_TX0_D2N, MIPI_DSI_TX0_D2P, MIPI_DSI_TX0_D3N, MIPI_DSI_TX0_D3P, MIPI_DSI_TX1_AVDD_0V9, MIPI_DSI_TX1_AVDD_1V8, MIPI_DSI_TX1_CLKN, MIPI_DSI_TX1_CLKP, MIPI_DSI_TX1_D0N, MIPI_DSI_TX1_D0P, MIPI_DSI_TX1_D1N, MIPI_DSI_TX1_D1P, MIPI_DSI_TX1_D2N, MIPI_DSI_TX1_D2P, MIPI_DSI_TX1_D3N, MIPI_DSI_TX1_D3P, MULTI_PHY0_REFCLKN, MULTI_PHY0_REFCLKP, MULTI_PHY1_REFCLKN, MULTI_PHY1_REFCLKP, MULTI_PHY_AVDD_0V9, MULTI_PHY_AVDD_1V8, OTP_VCC18, PCIE20_REFCLKN, PCIE20_REFCLKP, PCIE20_RXN, PCIE20_RXP, PCIE20_TXN, PCIE20_TXP, PCIE30_AVDD_0V9, PCIE30_AVDD_1V8, PCIE30_REFCLKN_IN, PCIE30_REFCLKP_IN, PCIE30_RESREF, PCIE30_RX0N, PCIE30_RX0P, PCIE30_RX1N, PCIE30_RX1P, PCIE30_TX0N, PCIE30_TX0P, PCIE30_TX1N, PCIE30_TX1P, PMIC_SLEEP, PMUIO1, PMUIO2, PMUPLL_AVDD_0V9, PMUPLL_AVDD_1V8, PMU_VDD_LOGIC_0V9, REFCLK_OUT, SARADC_AVDD_1V8, SARADC_VIN0, SARADC_VIN1, SARADC_VIN2, SARADC_VIN3, SARADC_VIN4, SARADC_VIN5, SARADC_VIN6, SARADC_VIN7, SDMMC0_CLK, SDMMC0_CMD, SDMMC0_D0, SDMMC0_D1, SDMMC0_D2, SDMMC0_D3, SDMMC0_DET, SDMMC1_CLK, SDMMC1_CMD, SDMMC1_D0, SDMMC1_D1, SDMMC1_D2, SDMMC1_D3, SDMMC1_DET, SDMMC1_PWREN, SYSPLL_AVDD_0V9, SYSPLL_AVDD_1V8, TSADC_SHUT, UART0_RX, UART0_TX, UART2_RX, UART2_TX, USB2_AVDD_0V9, USB2_AVDD_1V8, USB2_AVDD_3V3, USB2_HOST2_DM, USB2_HOST2_DP, USB2_HOST3_DM, USB2_HOST3_DP, USB3_AVDD_0V9, USB3_AVDD_1V8, USB3_AVDD_3V3, USB3_HOST1_DM, USB3_HOST1_DP, USB3_HOST1_SSRXN, USB3_HOST1_SSRXP, USB3_HOST1_SSTXN, USB3_HOST1_SSTXP, USB3_OTG0_DM, USB3_OTG0_DP, USB3_OTG0_ID, USB3_OTG0_SSRXN, USB3_OTG0_SSRXP, USB3_OTG0_SSTXN, USB3_OTG0_SSTXP, USB3_OTG0_VBUSDET, VCCIO1, VCCIO2, VCCIO3, VCCIO4, VCCIO5, VCCIO6, VCCIO7, VCC_DDR, VDD_CPU, VDD_GPU, VDD_LOGIC, VDD_NPU, XIN24M, XOUT24M, nPOR; removed none

Commit message: fixed netclasses
Other:
- sheet DDR Memory ports: added DDR_DM0_A, DDR_DM0_B, DDR_DM1_A, DDR_DM1_B, DDR_DQ0_A, DDR_DQ0_B, DDR_DQ10_A, DDR_DQ10_B, DDR_DQ11_A, DDR_DQ11_B, DDR_DQ12_A, DDR_DQ12_B, DDR_DQ13_A, DDR_DQ13_B, DDR_DQ14_A, DDR_DQ14_B, DDR_DQ15_A, DDR_DQ15_B, DDR_DQ1_A, DDR_DQ1_B, DDR_DQ2_A, DDR_DQ2_B, DDR_DQ3_A, DDR_DQ3_B, DDR_DQ4_A, DDR_DQ4_B, DDR_DQ5_A, DDR_DQ5_B, DDR_DQ6_A, DDR_DQ6_B, DDR_DQ7_A, DDR_DQ7_B, DDR_DQ8_A, DDR_DQ8_B, DDR_DQ9_A, DDR_DQ9_B, DDR_DQS0N_A, DDR_DQS0N_B, DDR_DQS0P_A, DDR_DQS0P_B, DDR_DQS1N_A, DDR_DQS1N_B, DDR_DQS1P_A, DDR_DQS1P_B, DDR_ZQ0, DDR_ZQ1, LPDDR4_CA0_A, LPDDR4_CA0_B, LPDDR4_CA1_A, LPDDR4_CA1_B, LPDDR4_CA2_A, LPDDR4_CA2_B, LPDDR4_CA3_A, LPDDR4_CA3_B, LPDDR4_CA4_A, LPDDR4_CA4_B, LPDDR4_CA5_A, LPDDR4_CA5_B, LPDDR4_CKE0_A, LPDDR4_CKE0_B, LPDDR4_CKE1_A, LPDDR4_CKE1_B, LPDDR4_CK_C_A, LPDDR4_CK_C_B, LPDDR4_CK_T_A, LPDDR4_CK_T_B, LPDDR4_CS0_A, LPDDR4_CS0_B, LPDDR4_CS1_A, LPDDR4_CS1_B, LPDDR4_ODT_CA_A, LPDDR4_ODT_CA_B, LPDDR4_RESET_N, VDD1_DDR, VDD2_DDR, VDDQ_DDR; removed none
- sheet SoC ports: added LPDDR4_CA0_A, LPDDR4_CA0_B, LPDDR4_CA1_A, LPDDR4_CA1_B, LPDDR4_CA2_A, LPDDR4_CA2_B, LPDDR4_CA3_A, LPDDR4_CA3_B, LPDDR4_CA4_A, LPDDR4_CA4_B, LPDDR4_CA5_A, LPDDR4_CA5_B, LPDDR4_CKE0_A, LPDDR4_CKE0_B, LPDDR4_CKE1_A, LPDDR4_CKE1_B, LPDDR4_CK_C_A, LPDDR4_CK_C_B, LPDDR4_CK_T_A, LPDDR4_CK_T_B, LPDDR4_CS0_A, LPDDR4_CS0_B, LPDDR4_CS1_A, LPDDR4_CS1_B, LPDDR4_ODT1_CA_A, LPDDR4_ODT1_CA_B, LPDDR4_ODT_CA_A, LPDDR4_ODT_CA_B, LPDDR4_RESET_N; removed DDR4_A0, DDR4_A1, DDR4_A10, DDR4_A11, DDR4_A12, DDR4_A13, DDR4_A14_WEn, DDR4_A15_CASn, DDR4_A16_RASn, DDR4_A2, DDR4_A3, DDR4_A4, DDR4_A5, DDR4_A6, DDR4_A7, DDR4_A8, DDR4_A9, DDR4_ACTn, DDR4_BA0, DDR4_BA1, DDR4_BG0, DDR4_BG1, DDR4_CKE, DDR4_CLKN, DDR4_CLKP, DDR4_CS0n, DDR4_CS1n, DDR4_ODT0, DDR4_ODT1, DDR4_RESETn

Commit message: display sheet
Other:
- sheet Display ports: added CSCL_GPIO3, DP1_AUX_N, DP1_AUX_P, DP1_HPD, DP1_TX0_N, DP1_TX0_P, DP1_TX1_N, DP1_TX1_P, DP1_TX2_N, DP1_TX2_P, DP1_TX3_N, DP1_TX3_P, EDP_TX_AUXN, EDP_TX_AUXP, EDP_TX_D0N, EDP_TX_D0P, EDP_TX_D1N, EDP_TX_D1P, EDP_TX_D2N, EDP_TX_D2P, EDP_TX_D3N, EDP_TX_D3P, HDMI_CEC, HDMI_CLK_N, HDMI_CLK_P, HDMI_DDC_SCL, HDMI_DDC_SDA, HDMI_HPD, HDMI_TX0_N, HDMI_TX0_P, HDMI_TX1_N, HDMI_TX1_P, HDMI_TX2_N, HDMI_TX2_P, IT6505_INT, IT6505_RST_N, IT6505_SCL, IT6505_SDA, LCDC_D0, LCDC_D1, LCDC_D10, LCDC_D11, LCDC_D12, LCDC_D13, LCDC_D14, LCDC_D15, LCDC_D16, LCDC_D17, LCDC_D18, LCDC_D19, LCDC_D2, LCDC_D20, LCDC_D21, LCDC_D22, LCDC_D23, LCDC_D3, LCDC_D4, LCDC_D5, LCDC_D6, LCDC_D7, LCDC_D8, LCDC_D9, LCDC_DCLK, LCDC_DEN, LCDC_HSYNC, LCDC_VSYNC, LT8711_INT, LT8711_RST_N, LT8711_SDA, USB_C_HDMI_CC1, USB_C_HDMI_CC2, USB_C_HDMI_CC2B, USB_C_HDMI_HPD, USB_C_HDMI_USB0_DN, USB_C_HDMI_USB0_DP, USB_C_HDMI_USB1_DN, USB_C_HDMI_USB1_DP, USB_C_HDMI_USB2_DN, USB_C_HDMI_USB2_DP, VBUS_HDMI, VCC1V2_DISP, VCC1V8_DISP, VCC3V3_DISP, VCC5V0; removed none
- sheet Storage ports: added EMMC_CLK, EMMC_CMD, EMMC_D0, EMMC_D1, EMMC_D2, EMMC_D3, EMMC_D4, EMMC_D5, EMMC_D6, EMMC_D7, EMMC_DATA_STROBE, EMMC_RSTN, SPI_FLASH_CLK, SPI_FLASH_CS, SPI_FLASH_HOLD, SPI_FLASH_MISO, SPI_FLASH_MOSI, SPI_FLASH_WP, VCC1V8_EMMC, VCC3V3_EMMC, VCC3V3_SYS; removed none

Commit message: USB Sheet
Other:
- sheet USB ports: added DP1_AUX_N, DP1_AUX_P, DP1_HPD, DP1_TX0_N, DP1_TX0_P, DP1_TX1_N, DP1_TX1_P, DP1_TX2_N, DP1_TX2_P, DP1_TX3_N, DP1_TX3_P, HDMI_CLK_N, HDMI_CLK_P, HDMI_TX0_N, HDMI_TX0_P, HDMI_TX1_N, HDMI_TX1_P, HDMI_TX2_N, HDMI_TX2_P, P1_PD_INT_N, P1_PD_SCL, P1_PD_SDA, P2_PD_INT_N, P2_PD_SCL, P2_PD_SDA, P3_MUX_OE, P3_MUX_SEL, P3_PD_INT_N, P3_PD_SCL, P3_PD_SDA, P4_MUX_OE, P4_MUX_SEL, P4_PD_INT_N, P4_PD_SCL, P4_PD_SDA, PCIE20_PERSTN, PCIE20_REFCLKN, PCIE20_REFCLKP, PCIE20_RXN, PCIE20_RXP, PCIE20_TXN, PCIE20_TXP, TUSB1064_SCL, TUSB1064_SDA, USB3_HOST1_DM, USB3_HOST1_DP, USB3_OTG0_DM, USB3_OTG0_DP, USB3_OTG0_SSRXN, USB3_OTG0_SSRXP, USB3_OTG0_SSTXN, USB3_OTG0_SSTXP, USB3_OTG0_VBUSDET, USB_C_HDMI_SBU1, USB_C_HDMI_SBU2; removed none

Commit message: GPIO and root sheet
Other:
- removed sheet DDR Memory
- added sheet LPDDR4X Memory (lpddr4x.kicad_sch)
- sheet Connectivity ports: added BT_HOST_WAKE, BT_REG_ON, BT_UART_CTS, BT_UART_RTS, BT_WAKE, SDMMC1_CLK, SDMMC1_CMD, SDMMC1_D0, SDMMC1_D1, SDMMC1_D2, SDMMC1_D3, UART0_RX, UART0_TX, WIFI_CLK32K, WIFI_HOST_WAKE, WIFI_REG_ON; removed none
- sheet GPIO and Expansion ports: added GPIO0_A5, GPIO0_A6, GPIO2_D0, GPIO3_C0, GPIO3_C1, GPIO3_C2, GPIO3_C3, GPIO3_C4, GPIO3_C5, GPIO3_C6, GPIO3_C7, GPIO3_D2, GPIO3_D3, GPIO3_D4, GPIO3_D5, GPIO3_D6, GPIO3_D7, GPIO4_A0, GPIO4_A1, GPIO4_A2, GPIO4_A3, GPIO4_A4, GPIO4_A5, GPIO4_A6, I2C3_SCL, I2C3_SDA, SARADC_VIN0, SDMMC0_CLK, SDMMC0_CMD, SDMMC0_D0, SDMMC0_D1, SDMMC0_D2, SDMMC0_D3, SDMMC0_DET, UART2_RX, UART2_TX, nPOR; removed none

Commit message: root sheet changes
Other:
- title: (none) -> Ganesh Pi
