File: usb.kicad_sch (KiCad schematic)
At the start: 0 parts

Commit message: USB Sheet
Parts:
- added C1, C17, C18, C19, C2, C20, C21, C22, C23, C24, C25, C26, C27, C28, C29, C3, C30, C4, C45, C48, C56, C57, C58: 100nF, symbol Device:C
- added C10, C11, C12, C13, C14, C15, C16, C9: 10uF, symbol Device:C
- added C46, C47: 20pF, symbol Device:C
- added C5, C6, C7, C8: 1uF, symbol Device:C
- added J1, J2, J3, J4: USB_C_Receptacle, symbol Connector:USB_C_Receptacle
- added R1, R2, R3: 10k, symbol Device:R
- added R4, R5: 100k, symbol Device:R
- added R6: 12k, symbol Device:R
- added U1: FUSB302BMPX, Package_DFN_QFN:WQFN-14-1EP_2.5x2.5mm_P0.5mm_EP1.45x1.45mm, symbol Interface_USB:FUSB302BMPX
- added U10, U11, U12, U3: NCP380HMU05AATBG_C463144, NCP380HMU05AATBG:UDFN-6_L2.0-W2.0-P0.65-BL-EP_MICROCHIP_MT, symbol NCP380HMU05AATBG:NCP380HMU05AATBG_C463144
- added U2, U9: HD3SS215RTQR, HD3SS215RTQR:HVQFN-56_L8.0-W8.0-P0.50-TL-EP4.5, symbol HD3SS215RTQR:HD3SS215RTQR
- added U4: VL805, VL805:QFN-68_L8.0-W8.0-P0.40-BL-EP6.2, symbol VL805:VL805
- added U5: FUSB302B10MPX, Package_DFN_QFN:WQFN-14-1EP_2.5x2.5mm_P0.5mm_EP1.45x1.45mm, symbol Interface_USB:FUSB302B10MPX
- added U6: TUSB1064RNQT, TUSB1064RNQT:WQFN-40_L6.0-W4.0-P0.40-TL-EP, symbol TUSB1064RNQT:TUSB1064RNQT
- added U7: FUSB302B01MPX, Package_DFN_QFN:WQFN-14-1EP_2.5x2.5mm_P0.5mm_EP1.45x1.45mm, symbol Interface_USB:FUSB302B01MPX
- added U8: FUSB302B11MPX, Package_DFN_QFN:WQFN-14-1EP_2.5x2.5mm_P0.5mm_EP1.45x1.45mm, symbol Interface_USB:FUSB302B11MPX
- added Y1: 25MHz, symbol Device:Crystal
Connections:
- new net: C47.2, U4.48 (SSXO)
- new net: R3.1, U4.31 (~{PONRST})
- new net: R6.2, U4.50 (SSREXT)
- new net: C5.2, U7.12 (VCONN), U7.13 (VCONN)
- new net: C17.2, U6.6 (VCC)
- new net: C1.2, U7.3 (VDD), U7.4 (VDD)
- new net: C3.2, U5.3 (VDD), U5.4 (VDD)
- new net: C2.2, U8.3 (VDD), U8.4 (VDD)
- new net: C4.2, U1.3 (VDD), U1.4 (VDD)
- new net: C8.2, U1.12 (VCONN), U1.13 (VCONN)
- new net: R2.2, U6.17 (I2C_EN)
- new net: C18.2, U6.20 (VCC)
- new net: C19.2, U6.28 (VCC)
- new net: R1.2, U6.29 (EN)
- new net: C7.2, U5.12 (VCONN), U5.13 (VCONN)
- new net: C6.2, U8.12 (VCONN), U8.13 (VCONN)
- new net +3V3: C21.1, C22.1, C23.1, C24.1, C25.1, C26.1, C27.1, C28.1, C29.1, C45.2, C48.2, C56.2, C57.2, C58.2, R1.1, R2.1, R3.2, U2.19 (VDD), U2.55 (VDD), U4.15 (VCCA33SS34), U4.23 (CCA33PEX), U4.29 (VDD), U4.32 (VSUS33), U4.45 (VDD), U4.46 (VSUS33), U4.49 (VCCA33SSM), U4.57 (VCCA33SS12), U4.6 (VCCA33SS34), U4.60 (VDD), U4.66 (VCCA33SS12), U4.9 (VDD), U9.19 (VDD), U9.55 (VDD)
- new net +5V: C11.1, C13.1, C15.1, C9.2, U10.6 (IN), U11.6 (IN), U12.6 (IN), U3.6 (IN)
- new net DP1_AUX_N: U6.27 (AUXn)
- new net DP1_AUX_P: U6.26 (AUXp)
- new net DP1_HPD: U6.32 (HPDIN)
- new net DP1_TX0_N: U6.39 (DP0n)
- new net DP1_TX0_P: U6.40 (DP0p)
- new net DP1_TX1_N: U6.36 (DP1n)
- new net DP1_TX1_P: U6.37 (DP1p)
- new net DP1_TX2_N: U6.33 (DP2n)
- new net DP1_TX2_P: U6.34 (DP2p)
- new net DP1_TX3_N: U6.30 (DP3n)
- new net DP1_TX3_P: U6.31 (DP3p)
- new net GND: C1.1, C10.2, C11.2, C12.2, C13.2, C14.2, C15.2, C16.2, C17.1, C18.1, C19.1, C2.1, C20.2, C21.2, C22.2, C23.2, C24.2, C25.2, C26.2, C27.2, C28.2, C29.2, C3.1, C30.2, C4.1, C45.1, C46.1, C47.1, C48.1, C5.1, C56.1, C57.1, C58.1, C6.1, C7.1, C8.1, C9.1, J1.A1 (GND), J1.A12 (GND), J1.B1 (GND), J1.B12 (GND), J2.A1 (GND), J2.A12 (GND), J2.B1 (GND), J2.B12 (GND), J3.A1 (GND), J3.A12 (GND), J3.B1 (GND), J3.B12 (GND), J4.A1 (GND), J4.A12 (GND), J4.B1 (GND), J4.B12 (GND), R5.2, R6.1, U1.15 (GND), U1.8 (GND), U1.9 (GND), U10.5 (GND), U10.7 (EP), U11.5 (GND), U11.7 (EP), U12.5 (GND), U12.7 (EP), U2.1 (AUX_SEL), U2.10 (GND), U2.33 (GND), U2.36 (GND), U2.39 (GND), U2.4 (GND), U2.46 (GND), U2.49 (GND), U2.52 (GND), U2.56 (DX_SEL), U2.57 (EP), U2.7 (GND), U3.5 (GND), U3.7 (EP), U4.51 (TESTEN), U4.69 (PAD), U5.15 (GND), U5.8 (GND), U5.9 (GND), U6.35 (DPEQ0/A1), U6.38 (SSEQ0/A0), U6.41 (EP), U7.15 (GND), U7.8 (GND), U7.9 (GND), U8.15 (GND), U8.8 (GND), U8.9 (GND), U9.1 (AUX_SEL), U9.10 (GND), U9.33 (GND), U9.36 (GND), U9.39 (GND), U9.4 (GND), U9.46 (GND), U9.49 (GND), U9.52 (GND), U9.56 (DX_SEL), U9.57 (EP), U9.7 (GND)
- new net HDMI_CLK_N: J2.B10 (RX1-)
- new net HDMI_CLK_P: J2.B11 (RX1+)
- new net HDMI_TX0_N: J2.B3 (TX2-)
- new net HDMI_TX0_P: J2.B2 (TX2+)
- new net HDMI_TX1_N: J2.A10 (RX2-)
- new net HDMI_TX1_P: J2.A11 (RX2+)
- new net HDMI_TX2_N: J2.A3 (TX1-)
- new net HDMI_TX2_P: J2.A2 (TX1+)
- new net P1_CC1: J1.A5 (CC1), U7.10 (CC1), U7.11 (CC1)
- new net P1_CC2: J1.B5 (CC2), U7.1 (CC2), U7.14 (CC2)
- new net P1_PD_INT_N: U7.5 (INT_N)
- new net P1_PD_SCL: U7.6 (SCL)
- new net P1_PD_SDA: U7.7 (SDA)
- new net P1_SBU1: J1.A8 (SBU1), U6.24 (SBU1)
- new net P1_SBU2: J1.B8 (SBU2), U6.25 (SBU2)
- new net P1_SSRX1N: J1.B10 (RX1-), U6.13 (RX1n)
- new net P1_SSRX1P: J1.B11 (RX1+), U6.12 (RX1p)
- new net P1_SSRX2N: J1.A10 (RX2-), U6.15 (RX2n)
- new net P1_SSRX2P: J1.A11 (RX2+), U6.16 (RX2p)
- new net P1_SSTX1N: J1.A3 (TX1-), U6.10 (TX1n)
- new net P1_SSTX1P: J1.A2 (TX1+), U6.9 (TX1p)
- new net P1_SSTX2N: J1.B3 (TX2-), U6.18 (TX2n)
- new net P1_SSTX2P: J1.B2 (TX2+), U6.19 (TX2p)
- new net P1_VBUS: C10.1, J1.A4 (VBUS), J1.A9 (VBUS), J1.B4 (VBUS), J1.B9 (VBUS), R4.1, U10.1 (OUT), U7.2 (VBUS)
- new net P1_VBUS_EN: U10.4 (EN), U4.44 (~{USBHRE1})
- new net P1_VBUS_OC: U10.3 (~{FLAG}), U4.43 (~{USBHRC1})
- new net P2_CC1: J2.A5 (CC1), U8.10 (CC1), U8.11 (CC1)
- new net P2_CC2: J2.B5 (CC2), U8.1 (CC2), U8.14 (CC2)
- new net P2_PD_INT_N: U8.5 (INT_N)
- new net P2_PD_SCL: U8.6 (SCL)
- new net P2_PD_SDA: U8.7 (SDA)
- new net P2_VBUS: C12.1, J2.A4 (VBUS), J2.A9 (VBUS), J2.B4 (VBUS), J2.B9 (VBUS), U11.1 (OUT), U8.2 (VBUS)
- new net P2_VBUS_EN: U11.4 (EN), U4.42 (~{USBHPE2})
- new net P2_VBUS_OC: U11.3 (~{FLAG}), U4.41 (~{USBHOC2})
- new net P3_CC1: J3.A5 (CC1), U5.10 (CC1), U5.11 (CC1)
- new net P3_CC2: J3.B5 (CC2), U5.1 (CC2), U5.14 (CC2)
- new net P3_MUX_OE: U2.43 (OE)
- new net P3_PD_INT_N: U5.5 (INT_N)
- new net P3_PD_SCL: U5.6 (SCL)
- new net P3_PD_SDA: U5.7 (SDA)
- new net P3_SSRX1N: J3.B10 (RX1-), U2.50 (DA1(N))
- new net P3_SSRX1P: J3.B11 (RX1+), U2.51 (DA1(P))
- new net P3_SSRX2N: J3.A10 (RX2-), U2.37 (DB1(N))
- new net P3_SSRX2P: J3.A11 (RX2+), U2.38 (DB1(P))
- new net P3_SSTX1N: J3.A3 (TX1-), U2.53 (DA0(N))
- new net P3_SSTX1P: J3.A2 (TX1+), U2.54 (DA0(P))
- new net P3_SSTX2N: J3.B3 (TX2-), U2.40 (DB0(N))
- new net P3_SSTX2P: J3.B2 (TX2+), U2.41 (DB0(P))
- new net P3_USB2_DM: J3.A7 (D-), J3.B7 (D-), U4.59 (USB2D1-)
- new net P3_USB2_DP: J3.A6 (D+), J3.B6 (D+), U4.58 (USB2D1+)
- new net P3_VBUS: C14.1, J3.A4 (VBUS), J3.A9 (VBUS), J3.B4 (VBUS), J3.B9 (VBUS), U12.1 (OUT), U5.2 (VBUS)
- new net P3_VBUS_EN: U12.4 (EN), U4.40 (~{USBHPE3})
- new net P3_VBUS_OC: U12.3 (~{FLAG}), U4.39 (~{USBHOC3})
- new net P4_CC1: J4.A5 (CC1), U1.10 (CC1), U1.11 (CC1)
- new net P4_CC2: J4.B5 (CC2), U1.1 (CC2), U1.14 (CC2)
- new net P4_MUX_OE: U9.43 (OE)
- new net P4_PD_INT_N: U1.5 (INT_N)
- new net P4_PD_SCL: U1.6 (SCL)
- new net P4_PD_SDA: U1.7 (SDA)
- new net P4_SSRX1N: J4.B10 (RX1-), U9.50 (DA1(N))
- new net P4_SSRX1P: J4.B11 (RX1+), U9.51 (DA1(P))
- new net P4_SSRX2N: J4.A10 (RX2-), U9.37 (DB1(N))
- new net P4_SSRX2P: J4.A11 (RX2+), U9.38 (DB1(P))
- new net P4_SSTX1N: J4.A3 (TX1-), U9.53 (DA0(N))
- new net P4_SSTX1P: J4.A2 (TX1+), U9.54 (DA0(P))
- new net P4_SSTX2N: J4.B3 (TX2-), U9.40 (DB0(N))
- new net P4_SSTX2P: J4.B2 (TX2+), U9.41 (DB0(P))
- new net P4_USB2_DM: J4.A7 (D-), J4.B7 (D-), U4.68 (USB2D2-)
- new net P4_USB2_DP: J4.A6 (D+), J4.B6 (D+), U4.67 (USB2D2+)
- new net P4_VBUS: C16.1, J4.A4 (VBUS), J4.A9 (VBUS), J4.B4 (VBUS), J4.B9 (VBUS), U1.2 (VBUS), U3.1 (OUT)
- new net P4_VBUS_EN: U3.4 (EN), U4.38 (~{USBHPE4})
- new net P4_VBUS_OC: U3.3 (~{FLAG}), U4.37 (~{USBHOC4})
- new net PCIE20_PERSTN: U4.19 (~{PEXRST})
- new net PCIE20_REFCLKN: U4.22 (PEXCLK-)
- new net PCIE20_REFCLKP: U4.21 (PEXCLK+)
- new net PCIE20_RXN: U4.28 (PEXRX0-)
- new net PCIE20_RXP: U4.27 (PEXRX0+)
- new net PCIE20_TXN: U4.25 (PEXTX0-)
- new net PCIE20_TXP: U4.24 (PEXTX0+)
- new net TUSB1064_SCL: U6.21 (FLIP/SCL)
- new net TUSB1064_SDA: U6.22 (CTL0/SDA)
- new net USB3_HOST1_DM: J2.A7 (D-), J2.B7 (D-)
- new net USB3_HOST1_DP: J2.A6 (D+), J2.B6 (D+)
- new net USB3_OTG0_DM: J1.A7 (D-), J1.B7 (D-)
- new net USB3_OTG0_DP: J1.A6 (D+), J1.B6 (D+)
- new net USB3_OTG0_SSRXN: U6.7 (SSTXn)
- new net USB3_OTG0_SSRXP: U6.8 (SSTXp)
- new net USB3_OTG0_SSTXN: U6.4 (SSRXn)
- new net USB3_OTG0_SSTXP: U6.5 (SSRXp)
- new net USB3_OTG0_VBUSDET: R4.2, R5.1
- new net USB_C_HDMI_SBU1: J2.B8 (SBU2)
- new net USB_C_HDMI_SBU2: J2.A8 (SBU1)
- new net VCCA10SSRX12: C30.1, U4.54 (VCCA10SSRX12), U4.63 (VCCA10SSRX12)
- new net VCCA10SSRX34: C20.1, U4.12 (VCCA10SSRX34), U4.3 (VCCA10SSRX34)
- new net VL805_DS1_SSRXN: U2.6 (DC1(N)), U4.56 (SSRX1-)
- new net VL805_DS1_SSRXP: U2.5 (DC1(P)), U4.55 (SSRX1+)
- new net VL805_DS1_SSTXN: U2.3 (DC0(N)), U4.53 (SSTX1-)
- new net VL805_DS1_SSTXP: U2.2 (DC0(P)), U4.52 (SSTX1+)
- new net VL805_DS2_SSRXN: U4.65 (SSRX2-), U9.6 (DC1(N))
- new net VL805_DS2_SSRXP: U4.64 (SSRX2+), U9.5 (DC1(P))
- new net VL805_DS2_SSTXN: U4.62 (SSTX2-), U9.3 (DC0(N))
- new net VL805_DS2_SSTXP: U4.61 (SSTX2+), U9.2 (DC0(P))
- new net VL805_XI: C46.2, U4.47 (SSXI), Y1.1
- new net VL805_XO: Y1.2
- no-connect marks 0 -> 94
Other:
- title: (none) -> USB ports

Commit message: GPIO and root sheet
Connections:
- net GND: now also J1.S1 (SHIELD), J2.S1 (SHIELD), J3.S1 (SHIELD), J4.S1 (SHIELD)
Other:
- moved on the sheet: C20, C21, C22, C23, C24, C25, C26, C27, C28, C29, C30, C45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

Commit message: root sheet changes
Parts:
- renumbered C58 to C100, C4 to C101, C8 to C102, C16 to C103, C17 to C67, C18 to C68, C9 to C69, C1 to C70, C5 to C71, C10 to C72, C19 to C73, C45 to C74, C20 to C75, C21 to C76, C11 to C77, C22 to C78, C23 to C79, C24 to C80, C2 to C81, C25 to C82, C6 to C83, C26 to C84, C27 to C85, C28 to C86, C12 to C87, C29 to C88, C30 to C89, C47 to C90, C46 to C91, C13 to C92, C48 to C93, C56 to C94, C3 to C95, C7 to C96, C14 to C97, C15 to C98, C57 to C99, R6 to R10, R2 to R5, R1 to R6, R4 to R7, R5 to R8, R3 to R9, U8 to U11, U4 to U12, U11 to U13, U5 to U14, U2 to U15, U12 to U16, U1 to U17, U9 to U18, U3 to U19, U7 to U8, U6 to U9, Y1 to Y4
